File: Backplane.kicad_sch (KiCad schematic)
At the start: 117 parts, among them J12 LOGIC, J13 LOGIC, J14 Conn_02x36_Odd_Even, U2 LM2991, U62 LT1086-ADJ, U63 LT1086-ADJ, U64 A32140DX, U65 SN74CBT3125, U66 SG-615P, U67 SN74FB2040, U68 MC100LVEL11, U7 LT1086-ADJ, U75 PCF8584, U76 74LS540

Commit message: Add component values, some more nets
Parts:
- C166, C167, C171, C172, C191, C192, C201: value ? -> 360pF
- C169, C170, C173, C174, C175, C193, C194, C195, C196, C197, C198, C199, C200, C84: value ? -> 0.047uF
- C85, C88, C89: value ? -> 1nF
Other:
- note added: "U21 D24"
- note added: "U21 D25"
- note added: "U22 D24"
- note added: "U22 D25"
- note added: "to U21 AE23, U22 AF24"
- note added: "to U21 AF24, U22 AE23"
- note removed: "to U21 AE23"
- note removed: "to U22 AE23"
- moved on the sheet: C167, C168, C170, C195, C196, C197, C199, R253, R255

Commit message: complete outer layers
Parts:
- removed U65: SN74CBT3125, Package_SO:SSOP-14_5.3x6.2mm_P0.65mm, symbol 74xx:74LS125
- added HS2, HS63, HS7: Heatsink_Pad, hp16717:HP_MINI_HEATSINK, symbol Mechanical:Heatsink_Pad
- added TP24, TP25: TestPoint, hp16717:HP_TP30, symbol Connector:TestPoint
- added U65: SN74CBT3125, hp16717:HP_SSOP-14_5.3x6.2mm_P0.65mm, symbol hp16717:SN74CBT3125
- C168, C78, C79: footprint Capacitor_Tantalum_SMD:CP_EIA-3528-21_Kemet-B -> hp16717:HP_CP_EIA-3528
- C176: footprint Capacitor_THT:CP_Axial_L30.0mm_D15.0mm_P35.00mm_Horizontal -> hp16717:HP_CP_Axial_L1300_D500_P1500_Horizontal
- C73, C74, C75, C76, C77, C80, C81, C82, C83: footprint Capacitor_Tantalum_SMD:CP_EIA-7343-31_Kemet-D -> hp16717:HP_CP_EIA-7343
- C86, C87: value 0.47uF -> 4.7uF; footprint Capacitor_Tantalum_SMD:CP_EIA-3528-21_Kemet-B -> hp16717:HP_CP_EIA-3528
- J12, J13: footprint Connector_PinHeader_2.54mm:PinHeader_2x10_P2.54mm_Vertical -> hp16717:HP_PinHeader_2x10_P2.54mm_Vertical
- U66: footprint Oscillator:Oscillator_SMD_SeikoEpson_SG8002JA-4Pin_14.0x8.7mm -> hp16717:HP_Oscillator_SMD_4Pin_14.0x8.7mm
- U75: footprint Package_SO:SOIC-20W_7.5x12.8mm_P1.27mm -> hp16717:HP_SOIC-20W_7.5x12.8mm_P1.27mm
- U76: value 74LS540 -> 74ABT540; footprint Package_SO:Infineon_SOIC-20W_7.6x12.8mm_P1.27mm -> hp16717:HP_SOIC-20W_7.5x12.8mm_P1.27mm
Connections:
- net +1V52: now also HS63.1
- net +3V3A: now also HS7.1
- net +5V: now also U65.14 (VCC)
- net -3V3: now also HS2.1
- net GND: now also U65.7 (GND)
- net I2C_POD1_2.SCL: now also U65.3 (1B)
- net I2C_POD1_2.SDA: now also U65.11 (4B)
- net I2C_POD3_4.SCL: now also U65.6 (2B)
- net I2C_POD3_4.SDA: now also U65.8 (3B)
- net POD12_I2C: now also U65.1 (1~{OE}), U65.13 (4~{OE})
- net POD34_I2C: now also U65.10 (3~{OE}), U65.4 (2~{OE})
- net U29_QSF: now also J12.6 (D13)
- net U39_QSF: now also J12.5 (D14)
- net ~{RAS3}: now also J12.4 (D15)
- net at R229.1, U75.2 (SDA/SDA_OUT): now also U65.12 (4A), U65.9 (3A)
- net at R228.1, U75.3 (SCL/SCL_OUT): now also U65.2 (1A), U65.5 (2A)
- net FA_UNK1: now reaches R230.2
- net FPGA_ASIC_XC1: now reaches R234.1, U64.145 (IO)
- net U22_FPGA0: now reaches RP17.1 (R1.1), U64.127 (IO)
- net U22_FPGA1: now reaches RP17.2 (R2.1), U64.128 (TCK/IO)
- net U22_FPGA2: now reaches RP17.3 (R3.1), U64.134 (IO)
- net U22_FPGA3: now reaches RP17.4 (R4.1), U64.158 (IO)
- net U21_FPGA0: now reaches RP17.5 (R5.1), U64.160 (IO)
- net U21_FPGA1: now reaches RP17.6 (R6.1), U64.161 (IO(WD))
- net U21_FPGA2: now reaches RP17.7 (R7.1), U64.162 (IO(WD))
- net U21_FPGA3: now reaches RP17.8 (R8.1), U64.163 (IO)
- net U22_FPGA4: now reaches RP10.1 (R1.1)
- net U21_FPGA4: now reaches RP10.2 (R2.1)
- net U22_FPGA5: now reaches RP10.3 (R3.1)
- net U21_FPGA5: now reaches RP10.4 (R4.1)
- net U22_FPGA6: now reaches RP10.5 (R5.1)
- net U21_FPGA6: now reaches RP10.6 (R6.1)
- net U22_FPGA7: now reaches RP10.7 (R7.1)
- net U21_FPGA7: now reaches RP10.8 (R8.1)
- net FPGA_ASIC_XC2: now reaches R233.1, U64.146 (IO)
- net U22_SYSCLK_N: now reaches R213.5 (R5.1)
- net U21_SYSCLK_N: now reaches R213.6 (R6.1)
- net U22_SYSCLK_P: now reaches R213.7 (R7.1)
- net U21_SYSCLK_P: now reaches R213.8 (R8.1)
- net ~{DAC_WR}: now reaches U64.147 (IO)
- net at U64.159 (SDI/IO): now also TP25.1
- net at U64.207 (DCLK/IO): now also TP24.1
- net 100M_SYSCLK renamed 100M_SYSCLK_P
- net 100M_SYSCLK2 renamed 100M_SYSCLK2_P
- net ~{100M_SYSCLK2} renamed 100M_SYSCLK2_N
- net ~{100M_SYSCLK} renamed 100M_SYSCLK_N
- no-connect marks 12 -> 18
Other:
- note removed: "FIXME: SYMBOL"
- note removed: "TODO: where does this go?"
- moved on the sheet: C166, C167, C168, C169, C170, C171, C173, C174, C175, C191, C192, C201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

Commit message: add test points
Parts:
- added TP100: CASR25, hp16717:HP_TP30, symbol Connector:TestPoint_Alt
- added TP101: CASR32, hp16717:HP_TP30, symbol Connector:TestPoint_Alt
- added TP102: CASR24, hp16717:HP_TP30, symbol Connector:TestPoint_Alt
- added TP103: CASR8, hp16717:HP_TP30, symbol Connector:TestPoint_Alt
- added TP104: CASR17, hp16717:HP_TP30, symbol Connector:TestPoint_Alt
- added TP105: CASR7, hp16717:HP_TP30, symbol Connector:TestPoint_Alt
- added TP1057, TP1061, TP1065, TP243, TP244, TP26, TP48, TP53, TP69, TP70: GND, hp16717:HP_TP30, symbol Connector:TestPoint_Alt
- added TP1058, TP1064, TP55, TP56, TP57, TP58, TP59, TP60: ?, hp16717:HP_TP30, symbol Connector:TestPoint_Alt
- added TP1059, TP1062: +3V3A, hp16717:HP_TP30, symbol Connector:TestPoint_Alt
- added TP106: CASR16, hp16717:HP_TP30, symbol Connector:TestPoint_Alt
- added TP1060: -1V7, hp16717:HP_TP30, symbol Connector:TestPoint_Alt
- added TP1063, TP160, TP204, TP206, TP247, TP71: +5V, hp16717:HP_TP30, symbol Connector:TestPoint_Alt
- added TP1066, TP1067, TP228, TP43, TP47, TP50: -3V3, hp16717:HP_TP30, symbol Connector:TestPoint_Alt
- added TP1068, TP44: -5V2, hp16717:HP_TP30, symbol Connector:TestPoint_Alt
- added TP107: RASR1, hp16717:HP_TP30, symbol Connector:TestPoint_Alt
- added TP108: RASR2, hp16717:HP_TP30, symbol Connector:TestPoint_Alt
- added TP109: RASR3, hp16717:HP_TP30, symbol Connector:TestPoint_Alt
- added TP110: IDB3, hp16717:HP_TP30, symbol Connector:TestPoint_Alt
- added TP1103: CMP_TEST_EN, hp16717:HP_TP30, symbol Connector:TestPoint_Alt
- added TP1108: RAS4, hp16717:HP_TP30, symbol Connector:TestPoint_Alt
- added TP111: RASR4, hp16717:HP_TP30, symbol Connector:TestPoint_Alt
- added TP112: CAS4, hp16717:HP_TP30, symbol Connector:TestPoint_Alt
- added TP113: CAS27, hp16717:HP_TP30, symbol Connector:TestPoint_Alt
- added TP114: CAS19, hp16717:HP_TP30, symbol Connector:TestPoint_Alt
- added TP115: IDB8, hp16717:HP_TP30, symbol Connector:TestPoint_Alt
- added TP116: IDB9, hp16717:HP_TP30, symbol Connector:TestPoint_Alt
- added TP117: IDB10, hp16717:HP_TP30, symbol Connector:TestPoint_Alt
- added TP118: IDB11, hp16717:HP_TP30, symbol Connector:TestPoint_Alt
- added TP119: IDB12, hp16717:HP_TP30, symbol Connector:TestPoint_Alt
- added TP120: IDB13, hp16717:HP_TP30, symbol Connector:TestPoint_Alt
- added TP121: IDB14, hp16717:HP_TP30, symbol Connector:TestPoint_Alt
- added TP122: IDB15, hp16717:HP_TP30, symbol Connector:TestPoint_Alt
- added TP123: CAS26, hp16717:HP_TP30, symbol Connector:TestPoint_Alt
- added TP124: CAS18, hp16717:HP_TP30, symbol Connector:TestPoint_Alt
- added TP125, TP130: CAS21, hp16717:HP_TP30, symbol Connector:TestPoint_Alt
- added TP126: CAS10, hp16717:HP_TP30, symbol Connector:TestPoint_Alt
- added TP127: CAS0, hp16717:HP_TP30, symbol Connector:TestPoint_Alt
- added TP128: CAS9, hp16717:HP_TP30, symbol Connector:TestPoint_Alt
- added TP129: CAS29, hp16717:HP_TP30, symbol Connector:TestPoint_Alt
- added TP131: CAS28, hp16717:HP_TP30, symbol Connector:TestPoint_Alt
- added TP132: CAS20, hp16717:HP_TP30, symbol Connector:TestPoint_Alt
- added TP133: CAS3, hp16717:HP_TP30, symbol Connector:TestPoint_Alt
- added TP134: CAS12, hp16717:HP_TP30, symbol Connector:TestPoint_Alt
- added TP135: CAS2, hp16717:HP_TP30, symbol Connector:TestPoint_Alt
- added TP136: CAS11, hp16717:HP_TP30, symbol Connector:TestPoint_Alt
- added TP137: CAS13, hp16717:HP_TP30, symbol Connector:TestPoint_Alt
- added TP138: CAS31, hp16717:HP_TP30, symbol Connector:TestPoint_Alt
- added TP139: CAS23, hp16717:HP_TP30, symbol Connector:TestPoint_Alt
- added TP140: CAS30, hp16717:HP_TP30, symbol Connector:TestPoint_Alt
- added TP141: CAS22, hp16717:HP_TP30, symbol Connector:TestPoint_Alt
- added TP142: CAS6, hp16717:HP_TP30, symbol Connector:TestPoint_Alt
- added TP143: CAS15, hp16717:HP_TP30, symbol Connector:TestPoint_Alt
- added TP144: CAS5, hp16717:HP_TP30, symbol Connector:TestPoint_Alt
- added TP145: CAS14, hp16717:HP_TP30, symbol Connector:TestPoint_Alt
- added TP146: CAS33, hp16717:HP_TP30, symbol Connector:TestPoint_Alt
- added TP147: CAS25, hp16717:HP_TP30, symbol Connector:TestPoint_Alt
- added TP148: CAS32, hp16717:HP_TP30, symbol Connector:TestPoint_Alt
- added TP149: CAS24, hp16717:HP_TP30, symbol Connector:TestPoint_Alt
- added TP150: CAS8, hp16717:HP_TP30, symbol Connector:TestPoint_Alt
- added TP151: CAS17, hp16717:HP_TP30, symbol Connector:TestPoint_Alt
- added TP152: CAS7, hp16717:HP_TP30, symbol Connector:TestPoint_Alt
- added TP153: CAS16, hp16717:HP_TP30, symbol Connector:TestPoint_Alt
- added TP154: PCF_A0, hp16717:HP_TP30, symbol Connector:TestPoint_Alt
- added TP155: PCF_CS, hp16717:HP_TP30, symbol Connector:TestPoint_Alt
- added TP156: PCF_RD, hp16717:HP_TP30, symbol Connector:TestPoint_Alt
- added TP157: PCF_WR, hp16717:HP_TP30, symbol Connector:TestPoint_Alt
- added TP158: PCF_CLK, hp16717:HP_TP30, symbol Connector:TestPoint_Alt
- added TP159: SCL, hp16717:HP_TP30, symbol Connector:TestPoint_Alt
- added TP161: FA_UNK1_R, hp16717:HP_TP30, symbol Connector:TestPoint_Alt
- added TP162: PCF_RST, hp16717:HP_TP30, symbol Connector:TestPoint_Alt
- added TP163: XC2_R, hp16717:HP_TP30, symbol Connector:TestPoint_Alt
- added TP164: IDB_CLK_R, hp16717:HP_TP30, symbol Connector:TestPoint_Alt
- added TP165: U22_FPGA0, hp16717:HP_TP30, symbol Connector:TestPoint_Alt
- added TP166: U22_FPGA1, hp16717:HP_TP30, symbol Connector:TestPoint_Alt
- added TP167: U22_FPGA2, hp16717:HP_TP30, symbol Connector:TestPoint_Alt
- added TP168: U22_FPGA3, hp16717:HP_TP30, symbol Connector:TestPoint_Alt
- added TP169: U21_FPGA0, hp16717:HP_TP30, symbol Connector:TestPoint_Alt
- added TP170: U21_FPGA1, hp16717:HP_TP30, symbol Connector:TestPoint_Alt
- added TP171: U21_FPGA2, hp16717:HP_TP30, symbol Connector:TestPoint_Alt
- added TP172: U21_FPGA3, hp16717:HP_TP30, symbol Connector:TestPoint_Alt
- added TP173: U22_FPGA4, hp16717:HP_TP30, symbol Connector:TestPoint_Alt
- added TP174: U21_FPGA4, hp16717:HP_TP30, symbol Connector:TestPoint_Alt
- added TP175: U22_FPGA5, hp16717:HP_TP30, symbol Connector:TestPoint_Alt
- added TP176: U21_FPGA5, hp16717:HP_TP30, symbol Connector:TestPoint_Alt
- added TP177: U22_FPGA6, hp16717:HP_TP30, symbol Connector:TestPoint_Alt
- added TP178: U21_FPGA6, hp16717:HP_TP30, symbol Connector:TestPoint_Alt
- added TP179: U22_FPGA7, hp16717:HP_TP30, symbol Connector:TestPoint_Alt
- added TP180: U21_FPGA7, hp16717:HP_TP30, symbol Connector:TestPoint_Alt
- added TP181: FA_UNK1, hp16717:HP_TP30, symbol Connector:TestPoint_Alt
- added TP182: FPGA4R, hp16717:HP_TP30, symbol Connector:TestPoint_Alt
- added TP183: HBDI0, hp16717:HP_TP30, symbol Connector:TestPoint_Alt
- added TP184: HBDI1, hp16717:HP_TP30, symbol Connector:TestPoint_Alt
- added TP185: HBDI2, hp16717:HP_TP30, symbol Connector:TestPoint_Alt
- added TP186: HBDI3, hp16717:HP_TP30, symbol Connector:TestPoint_Alt
- added TP187: HBDI4, hp16717:HP_TP30, symbol Connector:TestPoint_Alt
- added TP188: HBDI5, hp16717:HP_TP30, symbol Connector:TestPoint_Alt
- added TP189: HBDI6, hp16717:HP_TP30, symbol Connector:TestPoint_Alt
- added TP190: HBDI7, hp16717:HP_TP30, symbol Connector:TestPoint_Alt
- added TP191: HBDO0, hp16717:HP_TP30, symbol Connector:TestPoint_Alt
- added TP192: HBDO1, hp16717:HP_TP30, symbol Connector:TestPoint_Alt
- added TP193: HBDO2, hp16717:HP_TP30, symbol Connector:TestPoint_Alt
- added TP194: HBDO3, hp16717:HP_TP30, symbol Connector:TestPoint_Alt
- added TP195: HBDO4, hp16717:HP_TP30, symbol Connector:TestPoint_Alt
- added TP196: HBDO5, hp16717:HP_TP30, symbol Connector:TestPoint_Alt
- added TP197: HBDO6, hp16717:HP_TP30, symbol Connector:TestPoint_Alt
- added TP198: HBDO7, hp16717:HP_TP30, symbol Connector:TestPoint_Alt
- added TP199: TZCS_R0, hp16717:HP_TP30, symbol Connector:TestPoint_Alt
- added TP200: TZCS_R1, hp16717:HP_TP30, symbol Connector:TestPoint_Alt
- added TP201: TZCS_R2, hp16717:HP_TP30, symbol Connector:TestPoint_Alt
- added TP202: TZCS_R3, hp16717:HP_TP30, symbol Connector:TestPoint_Alt
- added TP203: TZCS_R4, hp16717:HP_TP30, symbol Connector:TestPoint_Alt
- added TP205: +3V3, hp16717:HP_TP30, symbol Connector:TestPoint_Alt
- added TP207: 1V52, hp16717:HP_TP30, symbol Connector:TestPoint_Alt
- added TP208: HBDO0B, hp16717:HP_TP30, symbol Connector:TestPoint_Alt
- added TP209: HBDO1B, hp16717:HP_TP30, symbol Connector:TestPoint_Alt
- added TP210: HBDO2B, hp16717:HP_TP30, symbol Connector:TestPoint_Alt
- added TP211: HBDO3B, hp16717:HP_TP30, symbol Connector:TestPoint_Alt
- added TP212: HBDO4B, hp16717:HP_TP30, symbol Connector:TestPoint_Alt
- added TP213: HBDO5B, hp16717:HP_TP30, symbol Connector:TestPoint_Alt
- added TP214: HBDO6B, hp16717:HP_TP30, symbol Connector:TestPoint_Alt
- added TP215: HBDO7B, hp16717:HP_TP30, symbol Connector:TestPoint_Alt
- added TP216: U21_HBDO0, hp16717:HP_TP30, symbol Connector:TestPoint_Alt
- added TP217: U22_HBDO1, hp16717:HP_TP30, symbol Connector:TestPoint_Alt
- added TP218: U21_HBDO2, hp16717:HP_TP30, symbol Connector:TestPoint_Alt
- added TP219: U22_HBDO3, hp16717:HP_TP30, symbol Connector:TestPoint_Alt
- added TP220: U21_HBDO4, hp16717:HP_TP30, symbol Connector:TestPoint_Alt
- added TP221: U22_HBDO5, hp16717:HP_TP30, symbol Connector:TestPoint_Alt
- added TP222: U21_HBDO6, hp16717:HP_TP30, symbol Connector:TestPoint_Alt
- added TP223: U22_HBDO7, hp16717:HP_TP30, symbol Connector:TestPoint_Alt
- added TP224: CK0_P, hp16717:HP_TP30, symbol Connector:TestPoint_Alt
- added TP225: CK0_N, hp16717:HP_TP30, symbol Connector:TestPoint_Alt
- added TP226: CK1_N, hp16717:HP_TP30, symbol Connector:TestPoint_Alt
- added TP227: CK1_P, hp16717:HP_TP30, symbol Connector:TestPoint_Alt
- added TP229: CK1C_P, hp16717:HP_TP30, symbol Connector:TestPoint_Alt
- added TP230: CK1C_N, hp16717:HP_TP30, symbol Connector:TestPoint_Alt
- added TP231: 100M_SYSCLK2_N, hp16717:HP_TP30, symbol Connector:TestPoint_Alt
- added TP232: 100M_SYSCLK2_P, hp16717:HP_TP30, symbol Connector:TestPoint_Alt
- added TP233: U22_SYSCLK2_N, hp16717:HP_TP30, symbol Connector:TestPoint_Alt
- added TP234: U21_SYSCLK2_N, hp16717:HP_TP30, symbol Connector:TestPoint_Alt
- added TP235: U22_SYSCLK2_P, hp16717:HP_TP30, symbol Connector:TestPoint_Alt
- added TP236: U21_SYSCLK2_P, hp16717:HP_TP30, symbol Connector:TestPoint_Alt
- added TP237: CK_N, hp16717:HP_TP30, symbol Connector:TestPoint_Alt
- added TP238: CK_P, hp16717:HP_TP30, symbol Connector:TestPoint_Alt
- added TP239: ~{HBD2}, hp16717:HP_TP30, symbol Connector:TestPoint_Alt
- added TP240: ~{HBD4}, hp16717:HP_TP30, symbol Connector:TestPoint_Alt
- added TP241: ~{HBD6}, hp16717:HP_TP30, symbol Connector:TestPoint_Alt
- added TP242: U63_ADJ, hp16717:HP_TP30, symbol Connector:TestPoint_Alt
- added TP245: U62_ADJ, hp16717:HP_TP30, symbol Connector:TestPoint_Alt
- added TP246: XC1_R, hp16717:HP_TP30, symbol Connector:TestPoint_Alt
- added TP248: RAS2, hp16717:HP_TP30, symbol Connector:TestPoint_Alt
- added TP249: DAC_WR, hp16717:HP_TP30, symbol Connector:TestPoint_Alt
- added TP250, TP251, TP252: +2V1, hp16717:HP_TP30, symbol Connector:TestPoint_Alt
- added TP253: U21_HBDO1, hp16717:HP_TP30, symbol Connector:TestPoint_Alt
- added TP254: U21_HBDO3, hp16717:HP_TP30, symbol Connector:TestPoint_Alt
- added TP255: U21_HBDO5, hp16717:HP_TP30, symbol Connector:TestPoint_Alt
- added TP256: U21_HBDO7, hp16717:HP_TP30, symbol Connector:TestPoint_Alt
- added TP257: U22_HBDO0, hp16717:HP_TP30, symbol Connector:TestPoint_Alt
- added TP258: U22_HBDO2, hp16717:HP_TP30, symbol Connector:TestPoint_Alt
- added TP259: U22_HBDO4, hp16717:HP_TP30, symbol Connector:TestPoint_Alt
- added TP260: U22_HBDO6, hp16717:HP_TP30, symbol Connector:TestPoint_Alt
- added TP261: LM311_OUT, hp16717:HP_TP30, symbol Connector:TestPoint_Alt
- added TP264: IAB2, hp16717:HP_TP30, symbol Connector:TestPoint_Alt
- added TP265: IAB3, hp16717:HP_TP30, symbol Connector:TestPoint_Alt
- added TP266: IAB4, hp16717:HP_TP30, symbol Connector:TestPoint_Alt
- added TP269: IAB7, hp16717:HP_TP30, symbol Connector:TestPoint_Alt
- added TP27: +12V, hp16717:HP_TP30, symbol Connector:TestPoint_Alt
- added TP270: IAB8, hp16717:HP_TP30, symbol Connector:TestPoint_Alt
- added TP271: VRAM_SE, hp16717:HP_TP30, symbol Connector:TestPoint_Alt
- added TP28: -12V, hp16717:HP_TP30, symbol Connector:TestPoint_Alt
- added TP29: BD7, hp16717:HP_TP30, symbol Connector:TestPoint_Alt
- added TP30: BD5, hp16717:HP_TP30, symbol Connector:TestPoint_Alt
- added TP31: BD3, hp16717:HP_TP30, symbol Connector:TestPoint_Alt
- added TP32: BD1, hp16717:HP_TP30, symbol Connector:TestPoint_Alt
- added TP33: FP208, hp16717:HP_TP30, symbol Connector:TestPoint_Alt
- added TP34: BA5, hp16717:HP_TP30, symbol Connector:TestPoint_Alt
- added TP35: BA3, hp16717:HP_TP30, symbol Connector:TestPoint_Alt
- added TP36: BA1, hp16717:HP_TP30, symbol Connector:TestPoint_Alt
- added TP37: BR/~{W}, hp16717:HP_TP30, symbol Connector:TestPoint_Alt
- added TP38: ~{BSEL}, hp16717:HP_TP30, symbol Connector:TestPoint_Alt
- added TP39: FP190, hp16717:HP_TP30, symbol Connector:TestPoint_Alt
- added TP40: ~{HBD1}, hp16717:HP_TP30, symbol Connector:TestPoint_Alt
- added TP41: FP144, hp16717:HP_TP30, symbol Connector:TestPoint_Alt
- added TP42: 100M_SYSCLK_P, hp16717:HP_TP30, symbol Connector:TestPoint_Alt
- added TP45: 19M66_OE, hp16717:HP_TP30, symbol Connector:TestPoint_Alt
- added TP46: CLK_FPGA, hp16717:HP_TP30, symbol Connector:TestPoint_Alt
- added TP49: FPGA_MODE, hp16717:HP_TP30, symbol Connector:TestPoint_Alt
- added TP51: POD12_I2C, hp16717:HP_TP30, symbol Connector:TestPoint_Alt
- added TP52: POD34_I2C, hp16717:HP_TP30, symbol Connector:TestPoint_Alt
- added TP54: SDA, hp16717:HP_TP30, symbol Connector:TestPoint_Alt
- added TP61: CLKSEL1, hp16717:HP_TP30, symbol Connector:TestPoint_Alt
- added TP62: ~{CLKEN1}, hp16717:HP_TP30, symbol Connector:TestPoint_Alt
- added TP63: CLKSEL1_5V, hp16717:HP_TP30, symbol Connector:TestPoint_Alt
- added TP64: CONFIG1, hp16717:HP_TP30, symbol Connector:TestPoint_Alt
- added TP65: CONFIG2, hp16717:HP_TP30, symbol Connector:TestPoint_Alt
- added TP66: CONFIG3, hp16717:HP_TP30, symbol Connector:TestPoint_Alt
- added TP67: ~{CLKEN1_5V}, hp16717:HP_TP30, symbol Connector:TestPoint_Alt
- added TP68: ~{16717A}, hp16717:HP_TP30, symbol Connector:TestPoint_Alt
- added TP72: VFILT_R, hp16717:HP_TP30, symbol Connector:TestPoint_Alt
- added TP73: CASR19, hp16717:HP_TP30, symbol Connector:TestPoint_Alt
- added TP74: CASR26, hp16717:HP_TP30, symbol Connector:TestPoint_Alt
- added TP75: CASR18, hp16717:HP_TP30, symbol Connector:TestPoint_Alt
- added TP76, TP83: CASR21, hp16717:HP_TP30, symbol Connector:TestPoint_Alt
- added TP77: CASR10, hp16717:HP_TP30, symbol Connector:TestPoint_Alt
- added TP78: CASR0, hp16717:HP_TP30, symbol Connector:TestPoint_Alt
- added TP79: CASR9, hp16717:HP_TP30, symbol Connector:TestPoint_Alt
- added TP80: CASR29, hp16717:HP_TP30, symbol Connector:TestPoint_Alt
- added TP81: CASR4, hp16717:HP_TP30, symbol Connector:TestPoint_Alt
- added TP82: CASR27, hp16717:HP_TP30, symbol Connector:TestPoint_Alt
- added TP84: CASR28, hp16717:HP_TP30, symbol Connector:TestPoint_Alt
- added TP85: CASR20, hp16717:HP_TP30, symbol Connector:TestPoint_Alt
- added TP86: CASR3, hp16717:HP_TP30, symbol Connector:TestPoint_Alt
- added TP87: CASR12, hp16717:HP_TP30, symbol Connector:TestPoint_Alt
- added TP88: CASR2, hp16717:HP_TP30, symbol Connector:TestPoint_Alt
- added TP89: CASR11, hp16717:HP_TP30, symbol Connector:TestPoint_Alt
- added TP90: CASR13, hp16717:HP_TP30, symbol Connector:TestPoint_Alt
- added TP91: CASR31, hp16717:HP_TP30, symbol Connector:TestPoint_Alt
- added TP92: CASR23, hp16717:HP_TP30, symbol Connector:TestPoint_Alt
- added TP93: CASR30, hp16717:HP_TP30, symbol Connector:TestPoint_Alt
- added TP94: CASR22, hp16717:HP_TP30, symbol Connector:TestPoint_Alt
- added TP95: CASR6, hp16717:HP_TP30, symbol Connector:TestPoint_Alt
- added TP96: CASR15, hp16717:HP_TP30, symbol Connector:TestPoint_Alt
- added TP97: CASR5, hp16717:HP_TP30, symbol Connector:TestPoint_Alt
- added TP98: CASR14, hp16717:HP_TP30, symbol Connector:TestPoint_Alt
- added TP99: CASR33, hp16717:HP_TP30, symbol Connector:TestPoint_Alt
Connections:
- net +12V: now also TP27.1
- net +1V52: now also TP207.1
- net +2V1: now also TP250.1, TP251.1, TP252.1
- net +3V3: now also TP205.1
- net +3V3A: now also TP1059.1, TP1062.1
- net +5V: now also TP1063.1, TP160.1, TP204.1, TP206.1, TP247.1, TP71.1
- net -12V: now also TP28.1
- net -1V7: now also TP1060.1
- net -3V3: now also TP1066.1, TP1067.1, TP228.1, TP43.1, TP47.1, TP50.1
- net -5V2: now also TP1068.1, TP44.1
- net 100M_SYSCLK2_N: now also TP231.1
- net 100M_SYSCLK2_P: now also TP232.1
- net 100M_SYSCLK_P: now also TP42.1
- net BA1: now also TP36.1
- net BA3: now also TP35.1
- net BA5: now also TP34.1
- net BD1: now also TP32.1
- net BD3: now also TP31.1
- net BD5: now also TP30.1
- net BD7: now also TP29.1
- net BR/~{W}: now also TP37.1
- net CLKSEL1: now also TP61.1
- net CLKSEL1_5V: now also TP63.1
- net CLK_FPGA: now also TP46.1
- net CONFIG1: now also TP64.1
- net CONFIG2: now also TP65.1
- net CONFIG3: now also TP66.1
- net FA_UNK1: now also TP181.1
- net FPGA_ASIC_XC1: now also TP246.1
- net FPGA_ASIC_XC2: now also TP163.1
- net FPGA_PIN144: now also TP41.1
- net FPGA_PIN190: now also TP39.1
- net FPGA_PIN208: now also TP33.1
- net GND: now also TP1057.1, TP1061.1, TP1065.1, TP243.1, TP244.1, TP26.1, TP48.1, TP53.1, TP69.1, TP70.1
- net HBDI0: now also TP183.1
- net HBDI1: now also TP184.1
- net HBDI2: now also TP185.1
- net HBDI3: now also TP186.1
- net HBDI4: now also TP187.1
- net HBDI5: now also TP188.1
- net HBDI6: now also TP189.1
- net HBDI7: now also TP190.1
- net HBDO0: now also TP191.1
- net HBDO1: now also TP192.1
- net HBDO2: now also TP193.1
- net HBDO3: now also TP194.1
- net HBDO4: now also TP195.1
- net HBDO5: now also TP196.1
- net HBDO6: now also TP197.1
- net HBDO7: now also TP198.1
- net IAB2: now also TP264.1
- net IAB3: now also TP265.1
- net IAB4: now also TP266.1
- net IAB7: now also TP269.1
- net IAB8: now also TP270.1
- net IDB10: now also TP117.1
- net IDB11: now also TP118.1
- net IDB12: now also TP119.1
- net IDB13: now also TP120.1
- net IDB14: now also TP121.1
- net IDB15: now also TP122.1
- net IDB3: now also TP110.1
- net IDB8: now also TP115.1
- net IDB9: now also TP116.1
- net LM311_OUT: now also TP261.1
- net PCF_A0: now also TP154.1
- net PCF_CLK: now also TP158.1
- net PCF_~{CS}: now also TP155.1
- net PCF_~{RD}: now also TP156.1
- net PCF_~{RST}: now also TP162.1
- net PCF_~{WR}: now also TP157.1
- net POD12_I2C: now also TP51.1
- net POD34_I2C: now also TP52.1
- net TZCS_R0: now also TP199.1
- net TZCS_R1: now also TP200.1
- net TZCS_R2: now also TP201.1
- net TZCS_R3: now also TP202.1
- net TZCS_R4: now also TP203.1
- net U21_FPGA0: now also TP169.1
- net U21_FPGA1: now also TP170.1
- net U21_FPGA2: now also TP171.1
- net U21_FPGA3: now also TP172.1
- net U21_FPGA4: now also TP174.1
- net U21_FPGA5: now also TP176.1
- net U21_FPGA6: now also TP178.1
- net U21_FPGA7: now also TP180.1
- net U21_HBDO0: now also TP216.1
- net U21_HBDO1: now also TP253.1
- net U21_HBDO2: now also TP218.1
- net U21_HBDO3: now also TP254.1
- net U21_HBDO4: now also TP220.1
- net U21_HBDO5: now also TP255.1
- net U21_HBDO6: now also TP222.1
- net U21_HBDO7: now also TP256.1
- net U21_SYSCLK_N: now also TP234.1
- net U21_SYSCLK_P: now also TP236.1
- net U22_FPGA0: now also TP165.1
- net U22_FPGA1: now also TP166.1
- net U22_FPGA2: now also TP167.1
- net U22_FPGA3: now also TP168.1
- net U22_FPGA4: now also TP173.1
- net U22_FPGA5: now also TP175.1
- net U22_FPGA6: now also TP177.1
- net U22_FPGA7: now also TP179.1
- net U22_HBDO0: now also TP257.1
- net U22_HBDO1: now also TP217.1
- net U22_HBDO2: now also TP258.1
- net U22_HBDO3: now also TP219.1
- net U22_HBDO4: now also TP259.1
- net U22_HBDO5: now also TP221.1
- net U22_HBDO6: now also TP260.1
- net U22_HBDO7: now also TP223.1
- net U22_SYSCLK_N: now also TP233.1
- net U22_SYSCLK_P: now also TP235.1
- net UNK_HPCLK1: now also TP60.1
- net UNK_HPCLK2: now also TP59.1
- net UNK_HPCLK3: now also TP58.1
- net UNK_HPCLK4: now also TP57.1
- net UNK_HPCLK5: now also TP56.1
- net UNK_HPCLK6: now also TP55.1
- net ~{16717A}: now also TP68.1
- net ~{BSEL}: now also TP38.1
- net ~{CAS0}: now also TP127.1
- net ~{CAS10}: now also TP126.1
- net ~{CAS11}: now also TP136.1
- net ~{CAS12}: now also TP134.1
- net ~{CAS13}: now also TP137.1
- net ~{CAS14}: now also TP145.1
- net ~{CAS15}: now also TP143.1
- net ~{CAS16}: now also TP153.1
- net ~{CAS17}: now also TP151.1
- net ~{CAS18}: now also TP124.1
- net ~{CAS19}: now also TP114.1
- net ~{CAS1}: now also TP125.1
- net ~{CAS20}: now also TP132.1
- net ~{CAS21}: now also TP130.1
- net ~{CAS22}: now also TP141.1
- net ~{CAS23}: now also TP139.1
- net ~{CAS24}: now also TP149.1
- net ~{CAS25}: now also TP147.1
- net ~{CAS26}: now also TP123.1
- net ~{CAS27}: now also TP113.1
- net ~{CAS28}: now also TP131.1
- net ~{CAS29}: now also TP129.1
- net ~{CAS2}: now also TP135.1
- net ~{CAS30}: now also TP140.1
- net ~{CAS31}: now also TP138.1
- net ~{CAS32}: now also TP148.1
- net ~{CAS33}: now also TP146.1
- net ~{CAS3}: now also TP133.1
- net ~{CAS4}: now also TP112.1
- net ~{CAS5}: now also TP144.1
- net ~{CAS6}: now also TP142.1
- net ~{CAS7}: now also TP152.1
- net ~{CAS8}: now also TP150.1
- net ~{CAS9}: now also TP128.1
- net ~{CASR0}: now also TP78.1
- net ~{CASR10}: now also TP77.1
- net ~{CASR11}: now also TP89.1
- net ~{CASR12}: now also TP87.1
- net ~{CASR13}: now also TP90.1
- net ~{CASR14}: now also TP98.1
- net ~{CASR15}: now also TP96.1
- net ~{CASR16}: now also TP106.1
- net ~{CASR17}: now also TP104.1
- net ~{CASR18}: now also TP75.1
- net ~{CASR19}: now also TP73.1
- net ~{CASR1}: now also TP76.1
- net ~{CASR20}: now also TP85.1
- net ~{CASR21}: now also TP83.1
- net ~{CASR22}: now also TP94.1
- net ~{CASR23}: now also TP92.1
- net ~{CASR24}: now also TP102.1
- net ~{CASR25}: now also TP100.1
- net ~{CASR26}: now also TP74.1
- net ~{CASR27}: now also TP82.1
- net ~{CASR28}: now also TP84.1
- net ~{CASR29}: now also TP80.1
- net ~{CASR2}: now also TP88.1
- net ~{CASR30}: now also TP93.1
- net ~{CASR31}: now also TP91.1
- net ~{CASR32}: now also TP101.1
- net ~{CASR33}: now also TP99.1
- net ~{CASR3}: now also TP86.1
- net ~{CASR4}: now also TP81.1
- net ~{CASR5}: now also TP97.1
- net ~{CASR6}: now also TP95.1
- net ~{CASR7}: now also TP105.1
- net ~{CASR8}: now also TP103.1
- net ~{CASR9}: now also TP79.1
- net ~{CLKEN1_5V}: now also TP67.1
- net ~{CLKEN1}: now also TP62.1
- net ~{CMP_TEST_EN}: now also TP1103.1
- net ~{DAC_WR}: now also TP249.1
- net ~{HBD1}: now also TP40.1
- net ~{HBD2}: now also TP239.1
- net ~{HBD4}: now also TP240.1
- net ~{HBD6}: now also TP241.1
- net ~{RAS2}: now also TP248.1
- net ~{RAS4}: now also TP1108.1
- net ~{VRAM_SE}: now also TP271.1
- net at C84.1, R151.1, R152.2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: now also TP1058.1
- net at R229.1, U65.12 (4A), U65.9 (3A)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: now also TP54.1
- net at R228.1, U65.2 (1A), U65.5 (2A)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: now also TP159.1
- net at R252.1, U64.3 (MODE): now also TP49.1
- net at R172.1, U68.7 (D): now also TP238.1
- net at R230.1, U64.177 (IO(WD)): now also TP161.1
- net ~{RAS1R}: now reaches R256.2, U64.58 (IO(WD))
- net ~{RAS1R}: now also TP107.1
- net at C175.1, R178.1, R213.10 (R7.2)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: now also TP230.1
- net at C175.2, R177.2, U68.4 (~{Q1}): now also TP226.1
- net at R154.1, R155.2, U2.1 (ADJ): now also TP1064.1
- net at RP16.7 (R7.1), RP9.10 (R7.2), U76.12 (Y6): now also TP214.1
- net at RP16.6 (R6.1), RP9.11 (R6.2), U76.13 (Y5): now also TP213.1
- net at RP16.5 (R5.1), RP9.12 (R5.2), U76.14 (Y4): now also TP212.1
- net at RP16.4 (R4.1), RP9.13 (R4.2), U76.15 (Y3): now also TP211.1
- net at RP16.3 (R3.1), RP9.14 (R3.2), U76.16 (Y2): now also TP210.1
- net at RP16.2 (R2.1), RP9.15 (R2.2), U76.17 (Y1): now also TP209.1
- net at RP16.1 (R1.1), RP9.16 (R1.2), U76.18 (Y0): now also TP208.1
- net at RP16.8 (R8.1), RP9.9 (R8.2), U76.11 (Y7): now also TP215.1
- net at C79.1, R149.1, R150.2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: now also TP242.1
- net at R175.2, R213.13 (R4.2), U68.2 (~{Q0}): now also TP225.1
- net at R174.2, R213.15 (R2.2), U68.1 (Q0): now also TP224.1
- net at C174.2, R176.2, U68.3 (Q1): now also TP227.1
- net at R173.1, U68.6 (~{D}): now also TP237.1
- net at C78.1, R147.1, R148.2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: now also TP245.1
- net ~{RAS4R}: now reaches R253.2, U64.62 (IO)
- net ~{RAS4R}: now also TP111.1
- net at R182.1, U66.1 (OE): now also TP45.1
- net at RP10.15 (R2.2), RP10.16 (R1.2), U64.135 (IO): now also TP182.1
- net at R232.1, U64.139 (IO): now also TP164.1
- net at C174.1, R179.1, R213.11 (R6.2)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: now also TP229.1
- net ~{RAS2R}: now reaches R255.2, U64.59 (IO)
- net ~{RAS2R}: now also TP108.1
- net at R214.2, U64.54 (TMS/IO): now also TP72.1
- net ~{RAS3R}: now reaches R254.2, U64.61 (IO)
- net ~{RAS3R}: now also TP109.1
Other:
- note added: "1GHZ PLL LOOP FILTER CTRL"
- moved on the sheet: C194, R253, R254, R255, R256
