File: Pod2.kicad_sch (KiCad schematic)
At the start: 156 parts, among them U3 1NB4-5036 Comparator, U4 1NB4-5036 Comparator

Commit message: Add component values, some more nets
Parts:
- C100, C102, C109, C125, C126, C127, C128, C129, C133, C134, C135, C136, C70, C72, C90, C91, C93, C94, C95, C96, C97, C99: value 330pF -> 360pF
- C103: value 330pF -> 1nF
- C156, C157, C158: value ? -> 0.047uF
Changed lines of the file:
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@@
 			)
 		)
-		(property "Value" "330pF"
+		(property "Value" "360pF"
 			(at 73.6663 293.37 90)
 			(effects
@@
 			)
 		)
-		(property "Value" "330pF"
+		(property "Value" "360pF"
 			(at 481.076 194.056 0)
 			(effects
@@
 			)
 		)
-		(property "Value" "330pF"
+		(property "Value" "360pF"
 			(at 210.82 82.5562 0)
 			(effects
@@
 			)
 		)
-		(property "Value" "?"
+		(property "Value" "0.047uF"
 			(at 208.534 203.454 0)
 			(effects
@@
 			)
 		)
-		(property "Value" "330pF"
+		(property "Value" "360pF"
 			(at 165.1 82.5562 0)
 			(effects
@@
 			)
 		)
-		(property "Value" "330pF"
+		(property "Value" "360pF"
 			(at 195.58 82.5562 0)
 			(effects
@@
 			)
 		)
-		(property "Value" "330pF"
+		(property "Value" "1nF"
 			(at 445.77 87.6362 0)
 			(effects
@@
 			)
 		)
-		(property "Value" "330pF"
+		(property "Value" "360pF"
 			(at 492.76 87.6362 0)
 			(effects
@@
 			)
 		)
-		(property "Value" "330pF"
+		(property "Value" "360pF"
 			(at 485.14 87.6362 0)
 			(effects
@@
 			)
 		)
-		(property "Value" "330pF"
+		(property "Value" "360pF"
 			(at 412.75 179.0762 0)
 			(effects
@@
 			)
 		)
-		(property "Value" "330pF"
+		(property "Value" "360pF"
 			(at 477.52 87.6362 0)
 			(effects
@@
 			)
 		)
-		(property "Value" "?"
+		(property "Value" "0.047uF"
 			(at 479.044 223.774 0)
 			(effects
@@
 			)
 		)
-		(property "Value" "330pF"
+		(property "Value" "360pF"
 			(at 218.44 82.5562 0)
 			(effects
@@
 			)
 		)
-		(property "Value" "330pF"
+		(property "Value" "360pF"
 			(at 173.99 179.0762 0)
 			(effects
@@
 			)
 		)
-		(property "Value" "330pF"
+		(property "Value" "360pF"
 			(at 508 87.6362 0)
 			(effects
@@
 			)
 		)
-		(property "Value" "330pF"
+		(property "Value" "360pF"
 			(at 195.834 179.324 0)
 			(effects
@@
 			)
 		)
-		(property "Value" "330pF"
+		(property "Value" "360pF"
 			(at 203.2 82.5562 0)
 			(effects
@@
 			)
 		)
-		(property "Value" "330pF"
+		(property "Value" "360pF"
 			(at 139.7 163.8362 0)
 			(effects
@@
 			)
 		)
-		(property "Value" "330pF"
+		(property "Value" "360pF"
 			(at 454.66 87.6362 0)
 			(effects
@@
 			)
 		)
-		(property "Value" "330pF"
+		(property "Value" "360pF"
 			(at 449.58 194.3162 0)
 			(effects
@@
 			)
 		)
-		(property "Value" "330pF"
+		(property "Value" "360pF"
 			(at 459.74 194.3162 0)
 			(effects
@@
 			)
 		)
-		(property "Value" "?"
+		(property "Value" "0.047uF"
 			(at 198.374 203.454 0)
 			(effects
@@
 			)
 		)
-		(property "Value" "330pF"
+		(property "Value" "360pF"
 			(at 205.486 178.816 0)
 			(effects
@@
 			)
 		)
-		(property "Value" "330pF"
+		(property "Value" "360pF"
 			(at 184.15 179.0762 0)
 			(effects
@@
 			)
 		)
-		(property "Value" "330pF"
+		(property "Value" "360pF"
 			(at 471.424 194.564 0)
 			(effects
@@
 			)
 		)
-		(property "Value" "330pF"
+		(property "Value" "360pF"
 			(at 500.38 87.6362 0)
 			(effects

Commit message: complete outer layers
Connections:
- net AP2_CLK renamed AP2_CLK_P
- net TZP2_CLK renamed TZP2_CLK_P
- net ~{AP2_CLK} renamed AP2_CLK_N
- net ~{TZP2_CLK} renamed TZP2_CLK_N
Changed lines of the file:
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@@
 		)
 	)
-	(label "~{TZP2_CLK}"
+	(label "TZP2_CLK_N"
 		(at 541.02 139.7 180)
 		(effects
@@
 		)
 	)
-	(label "~{AP2_CLK}"
+	(label "AP2_CLK_N"
 		(at 541.02 134.62 180)
 		(effects
@@
 		)
 	)
-	(label "TZP2_CLK"
+	(label "TZP2_CLK_P"
 		(at 541.02 127 180)
 		(effects
@@
 		)
 	)
-	(label "AP2_CLK"
+	(label "AP2_CLK_P"
 		(at 541.02 121.92 180)
 		(effects
@@
 		)
 	)
-	(hierarchical_label "~{TZP2_CLK}"
+	(hierarchical_label "TZP2_CLK_N"
 		(shape output)
 		(at 554.99 139.7 0)
@@
 		)
 	)
-	(hierarchical_label "~{AP2_CLK}"
+	(hierarchical_label "AP2_CLK_N"
 		(shape output)
 		(at 554.99 134.62 0)
@@
 		)
 	)
-	(hierarchical_label "AP2_CLK"
+	(hierarchical_label "AP2_CLK_P"
 		(shape output)
 		(at 554.99 121.92 0)
@@
 		)
 	)
-	(hierarchical_label "TZP2_CLK"
+	(hierarchical_label "TZP2_CLK_P"
 		(shape output)
 		(at 554.99 127 0)

Commit message: numerous small fixes, add plane and inner signal layers
Connections:
- net POD2A_VREF: now also R158.1, R159.2; no longer R156.1, R157.2
- net POD2B_VREF: now also R156.1, R157.2; no longer R158.1, R159.2
- net at U4.19 (2V1?): now also R131.1; no longer R126.3
- net at U3.19 (2V1?): now also R126.3; no longer R131.1
Other:
- moved on the sheet: R126B, R131A, R156, R157, R158, R159

Commit message: add test points
Parts:
- added TP1004, TP1017, TP1018, TP994: ?, hp16717:HP_TP30, symbol Connector:TestPoint_Alt
- added TP1019: -5V2, hp16717:HP_TP30, symbol Connector:TestPoint_Alt
- added TP977: POD2A_VREF, hp16717:HP_TP30, symbol Connector:TestPoint_Alt
- added TP978: POD2B_VREF, hp16717:HP_TP30, symbol Connector:TestPoint_Alt
- added TP985: POD2A_TZVREF, hp16717:HP_TP30, symbol Connector:TestPoint_Alt
- added TP986: PODBA_TZVREF, hp16717:HP_TP30, symbol Connector:TestPoint_Alt
- added TP995: -3V3, hp16717:HP_TP30, symbol Connector:TestPoint_Alt
- added TP996: +3V3, hp16717:HP_TP30, symbol Connector:TestPoint_Alt
Connections:
- net +3V3: now also TP996.1
- net -3V3: now also TP995.1
- net -5V2: now also TP1019.1
- net POD2A_TZVREF: now also TP985.1
- net POD2A_VREF: now also TP977.1
- net POD2B_TZVREF: now also TP986.1
- net POD2B_VREF: now also TP978.1
- net at R131.1, U4.19 (2V1?): now also TP1018.1
- net at R131.16, R159.1: now also TP1017.1
- net at R126.14, R157.1: now also TP994.1
- net at R126.3, U3.19 (2V1?): now also TP1004.1
