File: Pod4.kicad_sch (KiCad schematic)
At the start: 155 parts, among them U5 1NB4-5036 Comparator, U6 1NB4-5036 Comparator

Commit message: Add component values, some more nets
Parts:
- C322, C333, C334, C335, C337, C339, C341, C343, C344, C345, C347, C368, C369, C370, C371, C372, C374, C376, C377, C378, C379, C380: value 330pF -> 360pF
- C331, C332: value 10pF -> 2.2pF
- C342, C346: value ? -> 0.047uF
- C348: value 330pF -> 1nF
Other:
- note removed: "U21 pin K26"
Changed lines of the file:
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@@
 		)
 	)
-	(text "U21 pin K26"
-		(exclude_from_sim no)
-		(at 543.052 50.546 0)
-		(effects
-			(font
-				(size 1.27 1.27)
-			)
-		)
-	)
 	(junction
 		(at 346.71 55.88)
@@
 			)
 		)
-		(property "Value" "330pF"
+		(property "Value" "1nF"
 			(at 501.65 43.1862 0)
 			(effects
@@
 			)
 		)
-		(property "Value" "330pF"
+		(property "Value" "360pF"
 			(at 453.39 149.8662 0)
 			(effects
@@
 			)
 		)
-		(property "Value" "330pF"
+		(property "Value" "360pF"
 			(at 478.79 43.1862 0)
 			(effects
@@
 			)
 		)
-		(property "Value" "330pF"
+		(property "Value" "360pF"
 			(at 439.42 43.1862 0)
 			(effects
@@
 			)
 		)
-		(property "Value" "?"
+		(property "Value" "0.047uF"
 			(at 202.184 159.004 0)
 			(effects
@@
 			)
 		)
-		(property "Value" "330pF"
+		(property "Value" "360pF"
 			(at 406.4 134.6262 0)
 			(effects
@@
 			)
 		)
-		(property "Value" "330pF"
+		(property "Value" "360pF"
 			(at 486.41 43.1862 0)
 			(effects
@@
 			)
 		)
-		(property "Value" "330pF"
+		(property "Value" "360pF"
 			(at 196.85 38.1062 0)
 			(effects
@@
 			)
 		)
-		(property "Value" "330pF"
+		(property "Value" "360pF"
 			(at 167.64 134.6262 0)
 			(effects
@@
 			)
 		)
-		(property "Value" "330pF"
+		(property "Value" "360pF"
 			(at 133.35 119.3862 0)
 			(effects
@@
 			)
 		)
-		(property "Value" "330pF"
+		(property "Value" "360pF"
 			(at 465.074 150.114 0)
 			(effects
@@
 			)
 		)
-		(property "Value" "330pF"
+		(property "Value" "360pF"
 			(at 471.17 43.1862 0)
 			(effects
@@
 			)
 		)
-		(property "Value" "330pF"
+		(property "Value" "360pF"
 			(at 177.8 134.6262 0)
 			(effects
@@
 			)
 		)
-		(property "Value" "330pF"
+		(property "Value" "360pF"
 			(at 199.136 134.366 0)
 			(effects
@@
 			)
 		)
-		(property "Value" "330pF"
+		(property "Value" "360pF"
 			(at 448.31 43.1862 0)
 			(effects
@@
 			)
 		)
-		(property "Value" "330pF"
+		(property "Value" "360pF"
 			(at 494.03 43.1862 0)
 			(effects
@@
 			)
 		)
-		(property "Value" "?"
+		(property "Value" "0.047uF"
 			(at 192.024 159.004 0)
 			(effects
@@
 			)
 		)
-		(property "Value" "10pF"
+		(property "Value" "2.2pF"
 			(at 131.572 244.094 0)
 			(effects
@@
 			)
 		)
-		(property "Value" "10pF"
+		(property "Value" "2.2pF"
 			(at 130.556 269.494 0)
 			(effects
@@
 			)
 		)
-		(property "Value" "330pF"
+		(property "Value" "360pF"
 			(at 189.23 38.1062 0)
 			(effects
@@
 			)
 		)
-		(property "Value" "330pF"
+		(property "Value" "360pF"
 			(at 189.484 134.874 0)
 			(effects
@@
 			)
 		)
-		(property "Value" "330pF"
+		(property "Value" "360pF"
 			(at 443.23 149.8662 0)
 			(effects
@@
 			)
 		)
-		(property "Value" "330pF"
+		(property "Value" "360pF"
 			(at 204.47 38.1062 0)
 			(effects
@@
 			)
 		)
-		(property "Value" "330pF"
+		(property "Value" "360pF"
 			(at 158.75 38.1062 0)
 			(effects
@@
 			)
 		)
-		(property "Value" "330pF"
+		(property "Value" "360pF"
 			(at 474.726 149.606 0)
 			(effects
@@
 			)
 		)
-		(property "Value" "330pF"
+		(property "Value" "360pF"
 			(at 148.59 38.1062 0)
 			(effects
@@
 			)
 		)
-		(property "Value" "330pF"
+		(property "Value" "360pF"
 			(at 67.3163 248.92 90)
 			(effects

Commit message: complete outer layers
Connections:
- net AP4_CLK renamed AP4_CLK_P
- net TZP4_CLK renamed TZP4_CLK_P
- net ~{AP4_CLK} renamed AP4_CLK_N
- net ~{TZP4_CLK} renamed TZP4_CLK_N
Changed lines of the file:
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@@
 		)
 	)
-	(hierarchical_label "AP4_CLK"
+	(hierarchical_label "AP4_CLK_P"
 		(shape output)
 		(at 548.64 77.47 0)
@@
 		)
 	)
-	(hierarchical_label "~{TZP4_CLK}"
+	(hierarchical_label "TZP4_CLK_N"
 		(shape output)
 		(at 548.64 95.25 0)
@@
 		)
 	)
-	(hierarchical_label "~{AP4_CLK}"
+	(hierarchical_label "AP4_CLK_N"
 		(shape output)
 		(at 548.64 90.17 0)
@@
 		)
 	)
-	(hierarchical_label "TZP4_CLK"
+	(hierarchical_label "TZP4_CLK_P"
 		(shape output)
 		(at 548.64 82.55 0)

Commit message: add test points
Parts:
- added TP1031, TP1043, TP1044, TP1046: ?, hp16717:HP_TP30, symbol Connector:TestPoint_Alt
- added TP981: POD4A_VREF, hp16717:HP_TP30, symbol Connector:TestPoint_Alt
- added TP982: POD4B_VREF, hp16717:HP_TP30, symbol Connector:TestPoint_Alt
- added TP989: POD4B_TZVREF, hp16717:HP_TP30, symbol Connector:TestPoint_Alt
- added TP990: POD4A_TZVREF, hp16717:HP_TP30, symbol Connector:TestPoint_Alt
Connections:
- net POD4A_TZVREF: now also TP990.1
- net POD4A_VREF: now also TP981.1
- net POD4B_TZVREF: now also TP989.1
- net POD4B_VREF: now also TP982.1
- net at R134.1, U6.19 (2V1?): now also TP1044.1
- net at R128.14, R448.1: now also TP1046.1
- net at R128.3, U5.19 (2V1?): now also TP1031.1
- net at R134.16, R398.1: now also TP1043.1
