File: TimingZoom.kicad_sch (KiCad schematic)
At the start: 110 parts, among them J11 LOGIC, U10 1NB4-5040, U11 1NB4-5040, U12 1NB4-5040, U77 74LS08, U78 74LS08, U8 1NB4-5040, U9 1NB4-5040

Commit message: Add component values, some more nets
Parts:
- C229, C230, C232, C233, C235, C236, C237, C238, C239, C240, C241, C381, C383, C384, C385, C386, C387, C388, C389, C390, C391, C394, C395, C396, C397, C398, C399, C400, C401, C402, C403, C404, C407, C408, C409, C410, C411, C412, C413, C414, C415, C416, C417, C420, C421, C422, C423, C424, C425, C426, C427, C428, C429, C430, C433: value ? -> 1nF
- C231, C234, C392, C393, C405, C406, C418, C419, C431, C432, C460: value ? -> 360pF
- C434, C435, C436, C437, C438, C439, C441, C443, C444, C445, C446, C447, C448, C450, C451, C452, C453, C454, C455, C456, C457, C458, C459: value ? -> 100pF
- C440, C442, C449: value ? -> 390pF

Commit message: complete outer layers
Parts:
- J11: footprint Connector_PinHeader_2.54mm:PinHeader_2x10_P2.54mm_Vertical -> hp16717:HP_PinHeader_2x10_P2.54mm_Vertical
- RN10, RN11, RN12, RN13, RN9: footprint Resistor_SMD:R_Array_Convex_4x0603 -> hp16717:HP_R_Array_Convex_4x0603
- U77, U78: footprint Package_SO:SO-14_3.9x8.65mm_P1.27mm -> hp16717:HP_SO-14_3.9x8.65mm_P1.27mm
Connections:
- net TZCLKO1 renamed TZCLKO1_P
- net TZCLKO10 renamed TZCLKO10_P
- net TZCLKO2 renamed TZCLKO2_P
- net TZCLKO3 renamed TZCLKO3_P
- net TZCLKO4 renamed TZCLKO4_P
- net TZCLKO5 renamed TZCLKO5_P
- net TZCLKO6 renamed TZCLKO6_P
- net TZCLKO7 renamed TZCLKO7_P
- net TZCLKO8 renamed TZCLKO8_P
- net TZCLKO9 renamed TZCLKO9_P
- net TZP1_CLK renamed TZP1_CLK_P
- net TZP2_CLK renamed TZP2_CLK_P
- net TZP3_CLK renamed TZP3_CLK_P
- net TZP4_CLK renamed TZP4_CLK_P
- net ~{TZCLKO10} renamed TZCLKO10_N
- net ~{TZCLKO1} renamed TZCLKO1_N
- net ~{TZCLKO2} renamed TZCLKO2_N
- net ~{TZCLKO3} renamed TZCLKO3_N
- net ~{TZCLKO4} renamed TZCLKO4_N
- net ~{TZCLKO5} renamed TZCLKO5_N
- net ~{TZCLKO6} renamed TZCLKO6_N
- net ~{TZCLKO7} renamed TZCLKO7_N
- net ~{TZCLKO8} renamed TZCLKO8_N
- net ~{TZCLKO9} renamed TZCLKO9_N
- net ~{TZP1_CLK} renamed TZP1_CLK_N
- net ~{TZP2_CLK} renamed TZP2_CLK_N
- net ~{TZP3_CLK} renamed TZP3_CLK_N
- net ~{TZP4_CLK} renamed TZP4_CLK_N
Changed lines of the file:
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@@
 		)
 	)
-	(hierarchical_label "~{TZCLKO4}"
+	(hierarchical_label "TZCLKO4_N"
 		(shape input)
 		(at 52.07 156.21 180)
@@
 		)
 	)
-	(hierarchical_label "~{TZP4_CLK}"
+	(hierarchical_label "TZP4_CLK_N"
 		(shape input)
 		(at 127 143.51 180)
@@
 		)
 	)
-	(hierarchical_label "~{TZP1_CLK}"
+	(hierarchical_label "TZP1_CLK_N"
 		(shape input)
 		(at 127 275.59 180)
@@
 		)
 	)
-	(hierarchical_label "TZP1_CLK"
+	(hierarchical_label "TZP1_CLK_P"
 		(shape input)
 		(at 127 273.05 180)
@@
 		)
 	)
-	(hierarchical_label "~{TZCLKO6}"
+	(hierarchical_label "TZCLKO6_N"
 		(shape input)
 		(at 77.47 252.73 180)
@@
 		)
 	)
-	(hierarchical_label "~{TZP3_CLK}"
+	(hierarchical_label "TZP3_CLK_N"
 		(shape input)
 		(at 99.06 31.75 180)
@@
 		)
 	)
-	(hierarchical_label "~{TZCLKO3}"
+	(hierarchical_label "TZCLKO3_N"
 		(shape input)
 		(at 52.07 151.13 180)
@@
 		)
 	)
-	(hierarchical_label "TZCLKO5"
+	(hierarchical_label "TZCLKO5_P"
 		(shape input)
 		(at 77.47 245.11 180)
@@
 		)
 	)
-	(hierarchical_label "TZCLKO2"
+	(hierarchical_label "TZCLKO2_P"
 		(shape input)
 		(at 77.47 57.15 180)
@@
 		)
 	)
-	(hierarchical_label "TZCLKO4"
+	(hierarchical_label "TZCLKO4_P"
 		(shape input)
 		(at 52.07 153.67 180)
@@
 		)
 	)
-	(hierarchical_label "TZP2_CLK"
+	(hierarchical_label "TZP2_CLK_P"
 		(shape input)
 		(at 127 384.81 180)
@@
 		)
 	)
-	(hierarchical_label "~{TZCLKO10}"
+	(hierarchical_label "TZCLKO10_N"
 		(shape output)
 		(at 199.39 168.91 180)
@@
 		)
 	)
-	(hierarchical_label "TZCLKO9"
+	(hierarchical_label "TZCLKO9_P"
 		(shape output)
 		(at 199.39 161.29 180)
@@
 		)
 	)
-	(hierarchical_label "TZCLKO8"
+	(hierarchical_label "TZCLKO8_P"
 		(shape input)
 		(at 77.47 346.71 180)
@@
 		)
 	)
-	(hierarchical_label "~{TZCLKO5}"
+	(hierarchical_label "TZCLKO5_N"
 		(shape input)
 		(at 77.47 247.65 180)
@@
 		)
 	)
-	(hierarchical_label "TZCLKO3"
+	(hierarchical_label "TZCLKO3_P"
 		(shape input)
 		(at 52.07 148.59 180)
@@
 		)
 	)
-	(hierarchical_label "~{TZCLKO9}"
+	(hierarchical_label "TZCLKO9_N"
 		(shape output)
 		(at 199.39 163.83 180)
@@
 		)
 	)
-	(hierarchical_label "~{TZCLKO8}"
+	(hierarchical_label "TZCLKO8_N"
 		(shape input)
 		(at 77.47 349.25 180)
@@
 		)
 	)
-	(hierarchical_label "TZP3_CLK"
+	(hierarchical_label "TZP3_CLK_P"
 		(shape input)
 		(at 99.06 29.21 180)
@@
 		)
 	)
-	(hierarchical_label "~{TZCLKO2}"
+	(hierarchical_label "TZCLKO2_N"
 		(shape input)
 		(at 77.47 59.69 180)
@@
 		)
 	)
-	(hierarchical_label "TZCLKO10"
+	(hierarchical_label "TZCLKO10_P"
 		(shape output)
 		(at 199.39 166.37 180)
@@
 		)
 	)
-	(hierarchical_label "~{TZP2_CLK}"
+	(hierarchical_label "TZP2_CLK_N"
 		(shape input)
 		(at 127 387.35 180)
@@
 		)
 	)
-	(hierarchical_label "~{TZCLKO7}"
+	(hierarchical_label "TZCLKO7_N"
 		(shape input)
 		(at 77.47 344.17 180)
@@
 		)
 	)
-	(hierarchical_label "TZCLKO7"
+	(hierarchical_label "TZCLKO7_P"
 		(shape input)
 		(at 77.47 341.63 180)
@@
 		)
 	)
-	(hierarchical_label "TZCLKO6"
+	(hierarchical_label "TZCLKO6_P"
 		(shape input)
 		(at 77.47 250.19 180)
@@
 		)
 	)
-	(hierarchical_label "TZCLKO1"
+	(hierarchical_label "TZCLKO1_P"
 		(shape input)
 		(at 77.47 52.07 180)
@@
 		)
 	)
-	(hierarchical_label "TZP4_CLK"
+	(hierarchical_label "TZP4_CLK_P"
 		(shape input)
 		(at 127 140.97 180)
@@
 		)
 	)
-	(hierarchical_label "~{TZCLKO1}"
+	(hierarchical_label "TZCLKO1_N"
 		(shape input)
 		(at 77.47 54.61 180)
@@
 			)
 		)
-		(property "Footprint" "Package_SO:SO-14_3.9x8.65mm_P1.27mm"
+		(property "Footprint" "hp16717:HP_SO-14_3.9x8.65mm_P1.27mm"
 			(at 485.14 236.22 0)
 			(effects
@@
 			)
 		)
-		(property "Footprint" "Package_SO:SO-14_3.9x8.65mm_P1.27mm"
+		(property "Footprint" "hp16717:HP_SO-14_3.9x8.65mm_P1.27mm"
 			(at 168.91 149.86 0)
 			(effects
@@
 			)
 		)
-		(property "Footprint" "Resistor_SMD:R_Array_Convex_4x0603"
+		(property "Footprint" "hp16717:HP_R_Array_Convex_4x0603"
 			(at 95.885 356.87 90)
 			(effects
@@
 			)
 		)
-		(property "Footprint" "Package_SO:SO-14_3.9x8.65mm_P1.27mm"
+		(property "Footprint" "hp16717:HP_SO-14_3.9x8.65mm_P1.27mm"
 			(at 485.14 250.19 0)
 			(effects
@@
 			)
 		)
-		(property "Footprint" "Package_SO:SO-14_3.9x8.65mm_P1.27mm"
+		(property "Footprint" "hp16717:HP_SO-14_3.9x8.65mm_P1.27mm"
 			(at 290.83 168.91 0)
 			(effects
@@
 			)
 		)
-		(property "Footprint" "Connector_PinHeader_2.54mm:PinHeader_2x10_P2.54mm_Vertical"
+		(property "Footprint" "hp16717:HP_PinHeader_2x10_P2.54mm_Vertical"
 			(at 285.75 332.74 0)
 			(effects
@@
 			)
 		)
-		(property "Footprint" "Package_SO:SO-14_3.9x8.65mm_P1.27mm"
+		(property "Footprint" "hp16717:HP_SO-14_3.9x8.65mm_P1.27mm"
 			(at 485.14 222.25 0)
 			(effects
@@
 			)
 		)
-		(property "Footprint" "Package_SO:SO-14_3.9x8.65mm_P1.27mm"
+		(property "Footprint" "hp16717:HP_SO-14_3.9x8.65mm_P1.27mm"
 			(at 483.87 280.67 0)
 			(effects
@@
 			)
 		)
-		(property "Footprint" "Package_SO:SO-14_3.9x8.65mm_P1.27mm"
+		(property "Footprint" "hp16717:HP_SO-14_3.9x8.65mm_P1.27mm"
 			(at 168.91 50.8 0)
 			(effects
@@
 			)
 		)
-		(property "Footprint" "Resistor_SMD:R_Array_Convex_4x0603"
+		(property "Footprint" "hp16717:HP_R_Array_Convex_4x0603"
 			(at 95.885 260.35 90)
 			(effects
@@
 			)
 		)
-		(property "Footprint" "Resistor_SMD:R_Array_Convex_4x0603"
+		(property "Footprint" "hp16717:HP_R_Array_Convex_4x0603"
 			(at 95.885 67.31 90)
 			(effects
@@
 			)
 		)
-		(property "Footprint" "Package_SO:SO-14_3.9x8.65mm_P1.27mm"
+		(property "Footprint" "hp16717:HP_SO-14_3.9x8.65mm_P1.27mm"
 			(at 461.01 280.67 0)
 			(effects
@@
 			)
 		)
-		(property "Footprint" "Package_SO:SO-14_3.9x8.65mm_P1.27mm"
+		(property "Footprint" "hp16717:HP_SO-14_3.9x8.65mm_P1.27mm"
 			(at 166.37 345.44 0)
 			(effects
@@
 			)
 		)
-		(property "Footprint" "Package_SO:SO-14_3.9x8.65mm_P1.27mm"
+		(property "Footprint" "hp16717:HP_SO-14_3.9x8.65mm_P1.27mm"
 			(at 166.37 247.65 0)
 			(effects
@@
 			)
 		)
-		(property "Footprint" "Resistor_SMD:R_Array_Convex_4x0603"
+		(property "Footprint" "hp16717:HP_R_Array_Convex_4x0603"
 			(at 70.485 163.83 90)
 			(effects
@@
 			)
 		)
-		(property "Footprint" "Resistor_SMD:R_Array_Convex_4x0603"
+		(property "Footprint" "hp16717:HP_R_Array_Convex_4x0603"
 			(at 217.805 176.53 90)
 			(effects

Commit message: numerous small fixes, add plane and inner signal layers
Connections:
- net TZ_UNK5: no longer U12.80 (UNK)
- no-connect marks 23 -> 24
Changed lines of the file:
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@@
 	)
 	(junction
-		(at 279.4 134.62)
-		(diameter 0)
-		(color 0 0 0 0)
-	)
-	(junction
 		(at 222.25 353.06)
 		(diameter 0)
@@
 	)
 	(no_connect
+		(at 278.13 135.89)
+	)
+	(no_connect
 		(at 156.21 135.89)
 	)
@@
 	(wire
 		(pts
-			(xy 278.13 135.89) (xy 279.4 135.89)
-		)
-		(stroke
-			(width 0)
-			(type default)
-		)
-	)
-	(wire
-		(pts
 			(xy 83.82 363.22) (xy 83.82 361.95)
 		)
@@
 		)
 		(stroke
-			(width 0)
-			(type default)
-		)
-	)
-	(wire
-		(pts
-			(xy 279.4 134.62) (xy 279.4 135.89)
-		)
-		(stroke

Commit message: schematic tweaks, finish innermost layers
Connections:
- net GND: no longer U12.54 (GND)
- no-connect marks 24 -> 25
Changed lines of the file:
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@@
 	)
 	(junction
-		(at 528.32 69.85)
-		(diameter 0)
-		(color 0 0 0 0)
-	)
-	(junction
 		(at 561.34 74.93)
 		(diameter 0)
@@
 	)
 	(no_connect
+		(at 530.86 69.85)
+	)
+	(no_connect
 		(at 156.21 39.37)
 	)
@@
 	(wire
 		(pts
-			(xy 528.32 69.85) (xy 528.32 72.39)
+			(xy 528.32 67.31) (xy 528.32 72.39)
 		)
 		(stroke
@@
 	(wire
 		(pts
-			(xy 528.32 67.31) (xy 528.32 69.85)
-		)
-		(stroke
-			(width 0)
-			(type default)
-		)
-	)
-	(wire
-		(pts
 			(xy 312.42 41.91) (xy 314.96 41.91)
 		)
@@
 		)
 		(stroke
-			(width 0)
-			(type default)
-		)
-	)
-	(wire
-		(pts
-			(xy 528.32 69.85) (xy 530.86 69.85)
-		)
-		(stroke

Commit message: add test points
Parts:
- added TP902: TZLCK09_P, hp16717:HP_TP30, symbol Connector:TestPoint_Alt
- added TP903, TP904, TP905, TP906, TP907, TP908, TP909, TP910, TP911, TP912, TP913, TP914, TP915, TP916: +3V3, hp16717:HP_TP30, symbol Connector:TestPoint_Alt
- added TP917, TP918, TP919, TP920, TP921, TP922, TP923, TP924, TP925, TP926, TP927, TP928, TP929, TP930, TP931, TP932: GND, hp16717:HP_TP30, symbol Connector:TestPoint_Alt
- added TP933: TZCLKO1_N, hp16717:HP_TP30, symbol Connector:TestPoint_Alt
- added TP934: TZCLKO2_P, hp16717:HP_TP30, symbol Connector:TestPoint_Alt
- added TP935: TZCLKO3_N, hp16717:HP_TP30, symbol Connector:TestPoint_Alt
- added TP936: TZCLKO4_P, hp16717:HP_TP30, symbol Connector:TestPoint_Alt
- added TP937: TZCLKO5_N, hp16717:HP_TP30, symbol Connector:TestPoint_Alt
- added TP938: TZCLKO6_P, hp16717:HP_TP30, symbol Connector:TestPoint_Alt
- added TP939: TZCLKO7_N, hp16717:HP_TP30, symbol Connector:TestPoint_Alt
- added TP940: TZCLKO8_P, hp16717:HP_TP30, symbol Connector:TestPoint_Alt
- added TP941: TZP1_D0, hp16717:HP_TP30, symbol Connector:TestPoint_Alt
- added TP942: TZP1_D1, hp16717:HP_TP30, symbol Connector:TestPoint_Alt
- added TP943: TZP1_D2, hp16717:HP_TP30, symbol Connector:TestPoint_Alt
- added TP944: TZP1_D3, hp16717:HP_TP30, symbol Connector:TestPoint_Alt
- added TP945: TZP1_D4, hp16717:HP_TP30, symbol Connector:TestPoint_Alt
- added TP946: TZP1_D5, hp16717:HP_TP30, symbol Connector:TestPoint_Alt
- added TP947: TZP1_D6, hp16717:HP_TP30, symbol Connector:TestPoint_Alt
- added TP948: TZP1_D7, hp16717:HP_TP30, symbol Connector:TestPoint_Alt
- added TP949: TZP1_D8, hp16717:HP_TP30, symbol Connector:TestPoint_Alt
- added TP950: TZP1_D9, hp16717:HP_TP30, symbol Connector:TestPoint_Alt
- added TP951: TZP1_D10, hp16717:HP_TP30, symbol Connector:TestPoint_Alt
- added TP952: TZP1_D11, hp16717:HP_TP30, symbol Connector:TestPoint_Alt
- added TP953: TZP1_D12, hp16717:HP_TP30, symbol Connector:TestPoint_Alt
- added TP954: TZP1_D13, hp16717:HP_TP30, symbol Connector:TestPoint_Alt
- added TP955: TZP1_D14, hp16717:HP_TP30, symbol Connector:TestPoint_Alt
- added TP956: TZP1_D15, hp16717:HP_TP30, symbol Connector:TestPoint_Alt
- added TP957: TZP1_CLK_P, hp16717:HP_TP30, symbol Connector:TestPoint_Alt
- added TP958: TZP1_CLK_N, hp16717:HP_TP30, symbol Connector:TestPoint_Alt
- added TP959: TZP3_CLK_P, hp16717:HP_TP30, symbol Connector:TestPoint_Alt
- added TP961: TZP3_D0, hp16717:HP_TP30, symbol Connector:TestPoint_Alt
- added TP962: TZP3_D1, hp16717:HP_TP30, symbol Connector:TestPoint_Alt
- added TP963: TZP3_D2, hp16717:HP_TP30, symbol Connector:TestPoint_Alt
- added TP964: TZP3_D3, hp16717:HP_TP30, symbol Connector:TestPoint_Alt
- added TP966: TZP3_D5, hp16717:HP_TP30, symbol Connector:TestPoint_Alt
- added TP967: TZP3_D6, hp16717:HP_TP30, symbol Connector:TestPoint_Alt
- added TP968: TZP3_D7, hp16717:HP_TP30, symbol Connector:TestPoint_Alt
- added TP969: TZP3_D8, hp16717:HP_TP30, symbol Connector:TestPoint_Alt
- added TP970: TZP3_D9, hp16717:HP_TP30, symbol Connector:TestPoint_Alt
- added TP971: TZP3_D10, hp16717:HP_TP30, symbol Connector:TestPoint_Alt
- added TP972: TZP3_D11, hp16717:HP_TP30, symbol Connector:TestPoint_Alt
- added TP973: TZP3_D12, hp16717:HP_TP30, symbol Connector:TestPoint_Alt
- added TP974: TZP3_D13, hp16717:HP_TP30, symbol Connector:TestPoint_Alt
- added TP975: TZP3_D14, hp16717:HP_TP30, symbol Connector:TestPoint_Alt
- added TP976: TZP3_D15, hp16717:HP_TP30, symbol Connector:TestPoint_Alt
Connections:
- net +3V3: now also TP903.1, TP904.1, TP905.1, TP906.1, TP907.1, TP908.1, TP909.1, TP910.1, TP911.1, TP912.1, TP913.1, TP914.1, TP915.1, TP916.1
- net GND: now also TP917.1, TP918.1, TP919.1, TP920.1, TP921.1, TP922.1, TP923.1, TP924.1, TP925.1, TP926.1, TP927.1, TP928.1, TP929.1, TP930.1, TP931.1, TP932.1
- net TZCLKO1_N: now also TP933.1
- net TZCLKO2_P: now also TP934.1
- net TZCLKO3_N: now also TP935.1
- net TZCLKO4_P: now also TP936.1
- net TZCLKO5_N: now also TP937.1
- net TZCLKO6_P: now also TP938.1
- net TZCLKO7_N: now also TP939.1
- net TZCLKO8_P: now also TP940.1
- net TZCLKO9_P: now also TP902.1
- net TZP1_CLK_N: now also TP958.1
- net TZP1_CLK_P: now also TP957.1
- net TZP1_D0: now also TP941.1
- net TZP1_D1: now also TP942.1
- net TZP1_D10: now also TP951.1
- net TZP1_D11: now also TP952.1
- net TZP1_D12: now also TP953.1
- net TZP1_D13: now also TP954.1
- net TZP1_D14: now also TP955.1
- net TZP1_D15: now also TP956.1
- net TZP1_D2: now also TP943.1
- net TZP1_D3: now also TP944.1
- net TZP1_D4: now also TP945.1
- net TZP1_D5: now also TP946.1
- net TZP1_D6: now also TP947.1
- net TZP1_D7: now also TP948.1
- net TZP1_D8: now also TP949.1
- net TZP1_D9: now also TP950.1
- net TZP3_CLK_P: now also TP959.1
- net TZP3_D0: now also TP961.1
- net TZP3_D1: now also TP962.1
- net TZP3_D10: now also TP971.1
- net TZP3_D11: now also TP972.1
- net TZP3_D12: now also TP973.1
- net TZP3_D13: now also TP974.1
- net TZP3_D14: now also TP975.1
- net TZP3_D15: now also TP976.1
- net TZP3_D2: now also TP963.1
- net TZP3_D3: now also TP964.1
- net TZP3_D5: now also TP966.1
- net TZP3_D6: now also TP967.1
- net TZP3_D7: now also TP968.1
- net TZP3_D8: now also TP969.1
- net TZP3_D9: now also TP970.1
Other:
- moved on the sheet: C229, C230, C231, C232, C233, C234, C235, C236, C237, C238, C239, C240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
