File: HSInterconnect.kicad_sch (KiCad schematic)
At the start: 110 parts, among them J10 Conn_02x40_Odd_Even, J15 Conn_02x40_Odd_Even, J16 Conn_02x40_Odd_Even, J9 Conn_02x40_Odd_Even, Q1 MMBT3904, Q10 AT41511, Q11 AT41511, Q12 AT41511, Q13 AT41511, Q2 AT41511, Q3 AT41511, Q4 AT41511, Q5 AT41511, Q6 AT41511, Q7 AT41511, Q8 AT41511, Q9 AT41511, U17 MC100LVEL16, U18 MC100LVEL16, U19 MC100LVEL16, U20 MC100LVEL16, U23 MC100LVEL16, U24 MC100LVEL16

Commit message: Add component values, some more nets
Parts:
- C462, C463, C464, C465, C466, C476, C477, C478, C479, C480: value ? -> 3.3nF
- C471, C472, C473, C474: value ? -> 0.047uF
- C475: value ? -> 360pF
Changed lines of the file:
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@@
 			)
 		)
-		(property "Value" "?"
+		(property "Value" "3.3nF"
 			(at 524.51 267.9762 0)
 			(effects
@@
 			)
 		)
-		(property "Value" "?"
+		(property "Value" "3.3nF"
 			(at 549.91 267.9762 0)
 			(effects
@@
 			)
 		)
-		(property "Value" "?"
+		(property "Value" "3.3nF"
 			(at 542.29 267.9762 0)
 			(effects
@@
 			)
 		)
-		(property "Value" "?"
+		(property "Value" "0.047uF"
 			(at 191.77 246.3862 0)
 			(effects
@@
 			)
 		)
-		(property "Value" "?"
+		(property "Value" "0.047uF"
 			(at 173.99 246.3862 0)
 			(effects
@@
 			)
 		)
-		(property "Value" "?"
+		(property "Value" "3.3nF"
 			(at 408.94 76.2062 0)
 			(effects
@@
 			)
 		)
-		(property "Value" "?"
+		(property "Value" "0.047uF"
 			(at 163.83 246.3862 0)
 			(effects
@@
 			)
 		)
-		(property "Value" "?"
+		(property "Value" "3.3nF"
 			(at 203.2 99.0662 0)
 			(effects
@@
 			)
 		)
-		(property "Value" "?"
+		(property "Value" "3.3nF"
 			(at 383.54 76.2062 0)
 			(effects
@@
 			)
 		)
-		(property "Value" "?"
+		(property "Value" "360pF"
 			(at 209.55 223.5262 0)
 			(effects
@@
 			)
 		)
-		(property "Value" "?"
+		(property "Value" "3.3nF"
 			(at 401.32 76.2062 0)
 			(effects
@@
 			)
 		)
-		(property "Value" "?"
+		(property "Value" "3.3nF"
 			(at 392.43 76.2062 0)
 			(effects
@@
 			)
 		)
-		(property "Value" "?"
+		(property "Value" "0.047uF"
 			(at 182.88 246.3862 0)
 			(effects
@@
 			)
 		)
-		(property "Value" "?"
+		(property "Value" "3.3nF"
 			(at 219.71 287.0262 0)
 			(effects
@@
 			)
 		)
-		(property "Value" "?"
+		(property "Value" "3.3nF"
 			(at 533.4 267.9762 0)
 			(effects

Commit message: complete outer layers
Parts:
- C467, C468: footprint Capacitor_Tantalum_SMD:CP_EIA-7343-31_Kemet-D -> hp16717:HP_CP_EIA-7343
- C469: footprint Capacitor_Tantalum_SMD:CP_EIA-3528-21_Kemet-B -> hp16717:HP_CP_EIA-3528
- C470: value 0.47uF -> 4.7uF; footprint Capacitor_Tantalum_SMD:CP_EIA-3528-21_Kemet-B -> hp16717:HP_CP_EIA-3528
- Q1: footprint Active:SOT95P230X117-3 -> hp16717:HP_SOT95P230X117-3
- Q10, Q11, Q12, Q13, Q2, Q3, Q4, Q5, Q6, Q7, Q8, Q9: footprint Package_TO_SOT_SMD:SOT-143 -> hp16717:HP_SOT-143
Changed lines of the file:
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@@
 			)
 		)
-		(property "Footprint" "Package_TO_SOT_SMD:SOT-143"
+		(property "Footprint" "hp16717:HP_SOT-143"
 			(at 386.08 269.24 0)
 			(effects
@@
 			)
 		)
-		(property "Footprint" "Package_TO_SOT_SMD:SOT-143"
+		(property "Footprint" "hp16717:HP_SOT-143"
 			(at 242.57 81.28 0)
 			(effects
@@
 			)
 		)
-		(property "Footprint" "Package_TO_SOT_SMD:SOT-143"
+		(property "Footprint" "hp16717:HP_SOT-143"
 			(at 238.76 269.24 0)
 			(effects
@@
 			)
 		)
-		(property "Footprint" "Package_TO_SOT_SMD:SOT-143"
+		(property "Footprint" "hp16717:HP_SOT-143"
 			(at 259.08 269.24 0)
 			(effects
@@
 			)
 		)
-		(property "Footprint" "Capacitor_Tantalum_SMD:CP_EIA-3528-21_Kemet-B"
+		(property "Footprint" "hp16717:HP_CP_EIA-3528"
 			(at 181.61 222.25 0)
 			(effects
@@
 			)
 		)
-		(property "Value" "0.47uF"
+		(property "Value" "4.7uF"
 			(at 198.12 223.0881 0)
 			(effects
@@
 			)
 		)
-		(property "Footprint" "Capacitor_Tantalum_SMD:CP_EIA-3528-21_Kemet-B"
+		(property "Footprint" "hp16717:HP_CP_EIA-3528"
 			(at 195.58 222.25 0)
 			(effects
@@
 			)
 		)
-		(property "Footprint" "Package_TO_SOT_SMD:SOT-143"
+		(property "Footprint" "hp16717:HP_SOT-143"
 			(at 365.76 269.24 0)
 			(effects
@@
 			)
 		)
-		(property "Footprint" "Package_TO_SOT_SMD:SOT-143"
+		(property "Footprint" "hp16717:HP_SOT-143"
 			(at 222.25 81.28 0)
 			(effects
@@
 			)
 		)
-		(property "Footprint" "Capacitor_Tantalum_SMD:CP_EIA-7343-31_Kemet-D"
+		(property "Footprint" "hp16717:HP_CP_EIA-7343"
 			(at 161.29 222.25 0)
 			(effects
@@
 			)
 		)
-		(property "Footprint" "Package_TO_SOT_SMD:SOT-143"
+		(property "Footprint" "hp16717:HP_SOT-143"
 			(at 482.6 269.24 0)
 			(effects
@@
 			)
 		)
-		(property "Footprint" "Package_TO_SOT_SMD:SOT-143"
+		(property "Footprint" "hp16717:HP_SOT-143"
 			(at 502.92 269.24 0)
 			(effects
@@
 			)
 		)
-		(property "Footprint" "Package_TO_SOT_SMD:SOT-143"
+		(property "Footprint" "hp16717:HP_SOT-143"
 			(at 360.68 81.28 0)
 			(effects
@@
 			)
 		)
-		(property "Footprint" "Package_TO_SOT_SMD:SOT-143"
+		(property "Footprint" "hp16717:HP_SOT-143"
 			(at 340.36 81.28 0)
 			(effects
@@
 			)
 		)
-		(property "Footprint" "Package_TO_SOT_SMD:SOT-143"
+		(property "Footprint" "hp16717:HP_SOT-143"
 			(at 474.98 81.28 0)
 			(effects
@@
 			)
 		)
-		(property "Footprint" "Package_TO_SOT_SMD:SOT-143"
+		(property "Footprint" "hp16717:HP_SOT-143"
 			(at 454.66 81.28 0)
 			(effects
@@
 			)
 		)
-		(property "Footprint" "Active:SOT95P230X117-3"
+		(property "Footprint" "hp16717:HP_SOT95P230X117-3"
 			(at 204.47 282.575 0)
 			(effects
@@
 			)
 		)
-		(property "Footprint" "Capacitor_Tantalum_SMD:CP_EIA-7343-31_Kemet-D"
+		(property "Footprint" "hp16717:HP_CP_EIA-7343"
 			(at 171.45 222.25 0)
 			(effects

Commit message: schematic cleanup, arrange silk designators
Connections:
- net VBB_SI renamed U21_VBB_BI
- net U21_VBB_BI: no longer U18.4 (VBB)
- new net U22_VBB_BI: U18.4 (VBB)
Other:
- note added: "2 volts"
Changed lines of the file:
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@@
 		)
 	)
+	(text "2 volts"
+		(exclude_from_sim no)
+		(at 303.276 123.19 0)
+		(effects
+			(font
+				(size 1.27 1.27)
+			)
+		)
+	)
 	(text "U21 U26"
 		(exclude_from_sim no)
@@
 		)
 	)
+	(text "2 volts"
+		(exclude_from_sim no)
+		(at 321.056 310.896 0)
+		(effects
+			(font
+				(size 1.27 1.27)
+			)
+		)
+	)
 	(text "U22 R26"
 		(exclude_from_sim no)
@@
 	(wire
 		(pts
-			(xy 313.69 308.61) (xy 323.85 308.61)
+			(xy 313.69 308.61) (xy 327.66 308.61)
 		)
 		(stroke
@@
 	(wire
 		(pts
-			(xy 297.18 120.65) (xy 307.34 120.65)
+			(xy 297.18 120.65) (xy 309.88 120.65)
 		)
 		(stroke
@@
 		)
 	)
-	(label "VBB_SI"
-		(at 323.85 308.61 180)
+	(label "U21_VBB_BI"
+		(at 327.66 308.61 180)
 		(effects
 			(font
@@
 		)
 	)
-	(label "VBB_SI"
-		(at 307.34 120.65 180)
+	(label "U22_VBB_BI"
+		(at 309.88 120.65 180)
 		(effects
 			(font
@@
 		)
 	)
+	(hierarchical_label "U21_VBB_BI"
+		(shape output)
+		(at 327.66 308.61 0)
+		(effects
+			(font
+				(size 1.27 1.27)
+			)
+			(justify left)
+		)
+	)
 	(hierarchical_label "BI[1..6]"
 		(shape input)
@@
 		)
 	)
+	(hierarchical_label "U22_VBB_BI"
+		(shape output)
+		(at 309.88 120.65 0)
+		(effects
+			(font
+				(size 1.27 1.27)
+			)
+			(justify left)
+		)
+	)

Commit message: numerous small fixes, add plane and inner signal layers
Parts:
- removed Q1: MMBT3904, hp16717:HP_SOT95P230X117-3, symbol Transistor_BJT:MMBT3904
- added Q1: MMBT3906, hp16717:HP_SOT95P230X117-3, symbol Transistor_BJT:MMBT3906
Connections:
- net U21_BI18 is gone; now on net U21_BI8: R515.2
- net +3V3: now also Q1.2 (E)
- net ~{TERM_EN}: now also Q1.3 (C)
- net at R479.2: now also Q1.1 (B)
Other:
- moved on the sheet: R479
Changed lines of the file:
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@@
 	(wire
 		(pts
+			(xy 201.93 257.81) (xy 201.93 260.35)
+		)
+		(stroke
+			(width 0)
+			(type default)
+		)
+	)
+	(wire
+		(pts
 			(xy 34.29 267.97) (xy 45.72 267.97)
 		)
@@
 	(wire
 		(pts
+			(xy 201.93 270.51) (xy 201.93 271.78)
+		)
+		(stroke
+			(width 0)
+			(type default)
+		)
+	)
+	(wire
+		(pts
 			(xy 156.21 287.02) (xy 153.67 287.02)
 		)
@@
 	(wire
 		(pts
-			(xy 201.93 271.78) (xy 201.93 275.59)
-		)
-		(stroke
-			(width 0)
-			(type default)
-		)
-	)
-	(wire
-		(pts
 			(xy 242.57 90.17) (xy 242.57 97.79)
 		)
@@
 	(wire
 		(pts
+			(xy 191.77 265.43) (xy 194.31 265.43)
+		)
+		(stroke
+			(width 0)
+			(type default)
+		)
+	)
+	(wire
+		(pts
 			(xy 180.34 240.03) (xy 180.34 242.57)
 		)
@@
 		)
 	)
-	(label "U21_BI18"
+	(label "U21_BI8"
 		(at 553.72 109.22 180)
 		(effects
@@
 	(hierarchical_label "TERM_EN"
 		(shape input)
-		(at 189.23 280.67 180)
+		(at 186.69 265.43 180)
 		(effects
 			(font
@@
 	(symbol
 		(lib_id "Device:R_Small_US")
-		(at 191.77 280.67 90)
+		(at 189.23 265.43 90)
 		(mirror x)
 		(unit 1)
@@
 		(dnp no)
 		(property "Reference" "R479"
-			(at 189.23 275.59 90)
+			(at 186.69 260.35 90)
 			(effects
 				(font
@@
 		)
 		(property "Value" "1K"
-			(at 189.738 277.876 90)
+			(at 187.198 262.636 90)
 			(effects
 				(font
@@
 		)
 		(property "Footprint" "hp16717:HP_0805"
-			(at 191.77 280.67 0)
+			(at 189.23 265.43 0)
 			(effects
 				(font
@@
 		)
 		(property "Datasheet" "~"
-			(at 191.77 280.67 0)
+			(at 189.23 265.43 0)
 			(effects
 				(font
@@
 		)
 		(property "Description" "Resistor, small US symbol"
-			(at 191.77 280.67 0)
+			(at 189.23 265.43 0)
 			(effects
 				(font
@@
 	)
 	(symbol
+		(lib_id "Transistor_BJT:MMBT3906")
+		(at 199.39 265.43 0)
+		(mirror x)
+		(unit 1)
+		(exclude_from_sim no)
+		(in_bom yes)
+		(on_board yes)
+		(dnp no)
+		(property "Reference" "Q1"
+			(at 204.47 266.7001 0)
+			(effects
+				(font
+					(size 1.27 1.27)
+				)
+				(justify left)
+			)
+		)
+		(property "Value" "MMBT3906"
+			(at 204.47 264.1601 0)
+			(effects
+				(font
+					(size 1.27 1.27)
+				)
+				(justify left)
+			)
+		)
+		(property "Footprint" "hp16717:HP_SOT95P230X117-3"
+			(at 204.47 263.525 0)
+			(effects
+				(font
+					(size 1.27 1.27)
+					(italic yes)
+				)
+				(justify left)
+				(hide yes)
+			)
+		)
+		(property "Datasheet" "https://www.onsemi.com/pdf/datasheet/pzt3906-d.pdf"
+			(at 199.39 265.43 0)
+			(effects
+				(font
+					(size 1.27 1.27)
+				)
+				(justify left)
+				(hide yes)
+			)
+		)
+		(property "Description" "-0.2A Ic, -40V Vce, Small Signal PNP Transistor, SOT-23"
+			(at 199.39 265.43 0)
+			(effects
+				(font
+					(size 1.27 1.27)
+				)
+				(hide yes)
+			)
+		)
+		(pin "1"
+		)
+		(pin "2"
+		)
+		(pin "3"
+		)
+		(instances
+			(project ""
+				(path "/173036db-20dd-4729-b214-c668df2e6caa/d1d87433-66d8-4a4a-b366-85c8d9f4431f"
+					(reference "Q1")
+					(unit 1)
+				)
+			)
+		)
+	)
+	(symbol
 		(lib_id "power:GND")
 		(at 107.95 309.88 0)
@@
 	(symbol
 		(lib_id "power:GND")
-		(at 201.93 285.75 0)
-		(unit 1)
-		(exclude_from_sim no)
-		(in_bom yes)
-		(on_board yes)
-		(dnp no)
-		(fields_autoplaced yes)
-		(property "Reference" "#PWR0728"
-			(at 201.93 292.1 0)
-			(effects
-				(font
-					(size 1.27 1.27)
-				)
-				(hide yes)
-			)
-		)
-		(property "Value" "GND"
-			(at 201.93 290.83 0)
-			(effects
-				(font
-					(size 1.27 1.27)
-				)
-				(hide yes)
-			)
-		)
-		(property "Footprint" ""
-			(at 201.93 285.75 0)
-			(effects
-				(font
-					(size 1.27 1.27)
-				)
-				(hide yes)
-			)
-		)
-		(property "Datasheet" ""
-			(at 201.93 285.75 0)
-			(effects
-				(font
-					(size 1.27 1.27)
-				)
-				(hide yes)
-			)
-		)
-		(property "Description" "Power symbol creates a global label with name \"GND\" , ground"
-			(at 201.93 285.75 0)
-			(effects
-				(font
-					(size 1.27 1.27)
-				)
-				(hide yes)
-			)
-		)
-		(pin "1"
-		)
-		(instances
-			(project "hp16717"
-				(path "/173036db-20dd-4729-b214-c668df2e6caa/d1d87433-66d8-4a4a-b366-85c8d9f4431f"
-					(reference "#PWR0728")
-					(unit 1)
-				)
-			)
-		)
-	)
-	(symbol
-		(lib_id "power:GND")
 		(at 547.37 271.78 0)
 		(unit 1)
@@
 	)
 	(symbol
-		(lib_id "Transistor_BJT:MMBT3904")
-		(at 199.39 280.67 0)
+		(lib_id "power:+3V3")
+		(at 201.93 257.81 0)
+		(mirror y)
 		(unit 1)
 		(exclude_from_sim no)
@@
 		(on_board yes)
 		(dnp no)
-		(property "Reference" "Q1"
-			(at 204.47 281.9401 0)
+		(fields_autoplaced yes)
+		(property "Reference" "#PWR0728"
+			(at 201.93 261.62 0)
 			(effects
 				(font
 					(size 1.27 1.27)
 				)
-				(justify left)
+				(hide yes)
 			)
 		)
-		(property "Value" "MMBT3904"
-			(at 204.47 279.4001 0)
+		(property "Value" "+3V3"
+			(at 201.93 252.73 0)
 			(effects
 				(font
 					(size 1.27 1.27)
 				)
-				(justify left)
 			)
 		)
-		(property "Footprint" "hp16717:HP_SOT95P230X117-3"
-			(at 204.47 282.575 0)
+		(property "Footprint" ""
+			(at 201.93 257.81 0)
 			(effects
 				(font
 					(size 1.27 1.27)
-					(italic yes)
 				)
-				(justify left)
 				(hide yes)
 			)
 		)
-		(property "Datasheet" "https://www.onsemi.com/pdf/datasheet/pzt3904-d.pdf"
-			(at 199.39 280.67 0)
+		(property "Datasheet" ""
+			(at 201.93 257.81 0)
 			(effects
 				(font
 					(size 1.27 1.27)
 				)
-				(justify left)
 				(hide yes)
 			)
 		)
-		(property "Description" "0.2A Ic, 40V Vce, Small Signal NPN Transistor, SOT-23"
-			(at 199.39 280.67 0)
+		(property "Description" "Power symbol creates a global label with name \"+3V3\""
+			(at 201.93 257.81 0)
 			(effects
 				(font
@@
 			)
 		)
-		(pin "3"
-		)
 		(pin "1"
 		)
-		(pin "2"
-		)
 		(instances
 			(project "hp16717"
 				(path "/173036db-20dd-4729-b214-c668df2e6caa/d1d87433-66d8-4a4a-b366-85c8d9f4431f"
-					(reference "Q1")
+					(reference "#PWR0728")
 					(unit 1)
 				)

Commit message: add test points
Parts:
- added TP1101: U21_BI11, hp16717:HP_TP30, symbol Connector:TestPoint_Alt
- added TP1102: U21_BI12, hp16717:HP_TP30, symbol Connector:TestPoint_Alt
- added TP678: TERM_EN, hp16717:HP_TP30, symbol Connector:TestPoint_Alt
- added TP679, TP683, TP688, TP689, TP789, TP790, TP791, TP799: ?, hp16717:HP_TP30, symbol Connector:TestPoint_Alt
- added TP680: +3V3, hp16717:HP_TP30, symbol Connector:TestPoint_Alt
- added TP681: ~{TERM_EN}, hp16717:HP_TP30, symbol Connector:TestPoint_Alt
- added TP682: U22_BI7, hp16717:HP_TP30, symbol Connector:TestPoint_Alt
- added TP684: U22_BI12, hp16717:HP_TP30, symbol Connector:TestPoint_Alt
- added TP685: U22_BI8, hp16717:HP_TP30, symbol Connector:TestPoint_Alt
- added TP686: U22_BI10, hp16717:HP_TP30, symbol Connector:TestPoint_Alt
- added TP687: U22_BI9, hp16717:HP_TP30, symbol Connector:TestPoint_Alt
- added TP690, TP739, TP740, TP797, TP798: GND, hp16717:HP_TP30, symbol Connector:TestPoint_Alt
- added TP701: U22_VBB_BI, hp16717:HP_TP30, symbol Connector:TestPoint_Alt
- added TP705: U22_BI11, hp16717:HP_TP30, symbol Connector:TestPoint_Alt
- added TP713: SI0, hp16717:HP_TP30, symbol Connector:TestPoint_Alt
- added TP714: SI1, hp16717:HP_TP30, symbol Connector:TestPoint_Alt
- added TP715: SI2, hp16717:HP_TP30, symbol Connector:TestPoint_Alt
- added TP716: SI3, hp16717:HP_TP30, symbol Connector:TestPoint_Alt
- added TP717: SI4, hp16717:HP_TP30, symbol Connector:TestPoint_Alt
- added TP718: SI5, hp16717:HP_TP30, symbol Connector:TestPoint_Alt
- added TP719: SI6, hp16717:HP_TP30, symbol Connector:TestPoint_Alt
- added TP720: SI7, hp16717:HP_TP30, symbol Connector:TestPoint_Alt
- added TP721: SI8, hp16717:HP_TP30, symbol Connector:TestPoint_Alt
- added TP722: SI9, hp16717:HP_TP30, symbol Connector:TestPoint_Alt
- added TP723: SI10, hp16717:HP_TP30, symbol Connector:TestPoint_Alt
- added TP724: SI11, hp16717:HP_TP30, symbol Connector:TestPoint_Alt
- added TP725: SI12, hp16717:HP_TP30, symbol Connector:TestPoint_Alt
- added TP726: SI13, hp16717:HP_TP30, symbol Connector:TestPoint_Alt
- added TP727: SI14, hp16717:HP_TP30, symbol Connector:TestPoint_Alt
- added TP728: SI15, hp16717:HP_TP30, symbol Connector:TestPoint_Alt
- added TP729: SI16, hp16717:HP_TP30, symbol Connector:TestPoint_Alt
- added TP730: SI17, hp16717:HP_TP30, symbol Connector:TestPoint_Alt
- added TP731: SI18, hp16717:HP_TP30, symbol Connector:TestPoint_Alt
- added TP732: SI19, hp16717:HP_TP30, symbol Connector:TestPoint_Alt
- added TP733: SI20, hp16717:HP_TP30, symbol Connector:TestPoint_Alt
- added TP734: SI21, hp16717:HP_TP30, symbol Connector:TestPoint_Alt
- added TP735: SI22, hp16717:HP_TP30, symbol Connector:TestPoint_Alt
- added TP736: SI23, hp16717:HP_TP30, symbol Connector:TestPoint_Alt
- added TP737, TP738: +1V52, hp16717:HP_TP30, symbol Connector:TestPoint_Alt
- added TP745: NI0, hp16717:HP_TP30, symbol Connector:TestPoint_Alt
- added TP746: NI1, hp16717:HP_TP30, symbol Connector:TestPoint_Alt
- added TP747: NI2, hp16717:HP_TP30, symbol Connector:TestPoint_Alt
- added TP748: NI3, hp16717:HP_TP30, symbol Connector:TestPoint_Alt
- added TP749: NI4, hp16717:HP_TP30, symbol Connector:TestPoint_Alt
- added TP750: NI5, hp16717:HP_TP30, symbol Connector:TestPoint_Alt
- added TP751: NI6, hp16717:HP_TP30, symbol Connector:TestPoint_Alt
- added TP752: NI7, hp16717:HP_TP30, symbol Connector:TestPoint_Alt
- added TP753: NI8, hp16717:HP_TP30, symbol Connector:TestPoint_Alt
- added TP754: NI9, hp16717:HP_TP30, symbol Connector:TestPoint_Alt
- added TP755: NI10, hp16717:HP_TP30, symbol Connector:TestPoint_Alt
- added TP756: NI11, hp16717:HP_TP30, symbol Connector:TestPoint_Alt
- added TP757: NI12, hp16717:HP_TP30, symbol Connector:TestPoint_Alt
- added TP758: NI13, hp16717:HP_TP30, symbol Connector:TestPoint_Alt
- added TP759: NI14, hp16717:HP_TP30, symbol Connector:TestPoint_Alt
- added TP760: NI15, hp16717:HP_TP30, symbol Connector:TestPoint_Alt
- added TP761: NI16, hp16717:HP_TP30, symbol Connector:TestPoint_Alt
- added TP762: NI17, hp16717:HP_TP30, symbol Connector:TestPoint_Alt
- added TP763: NI18, hp16717:HP_TP30, symbol Connector:TestPoint_Alt
- added TP764: NI19, hp16717:HP_TP30, symbol Connector:TestPoint_Alt
- added TP765: NI20, hp16717:HP_TP30, symbol Connector:TestPoint_Alt
- added TP766: NI21, hp16717:HP_TP30, symbol Connector:TestPoint_Alt
- added TP767: NI22, hp16717:HP_TP30, symbol Connector:TestPoint_Alt
- added TP768: NI23, hp16717:HP_TP30, symbol Connector:TestPoint_Alt
- added TP778: U21_VBB_BI, hp16717:HP_TP30, symbol Connector:TestPoint_Alt
- added TP792: U21_BI1, hp16717:HP_TP30, symbol Connector:TestPoint_Alt
- added TP793: U21_BI3, hp16717:HP_TP30, symbol Connector:TestPoint_Alt
- added TP794: U21_BI4, hp16717:HP_TP30, symbol Connector:TestPoint_Alt
- added TP795: U21_BI5, hp16717:HP_TP30, symbol Connector:TestPoint_Alt
- added TP796: U21_BI6, hp16717:HP_TP30, symbol Connector:TestPoint_Alt
Connections:
- net +1V52: now also TP737.1, TP738.1
- net +3V3: now also TP680.1
- net GND: now also TP690.1, TP739.1, TP740.1, TP797.1, TP798.1
- net NI0: now also TP745.1
- net NI1: now also TP746.1
- net NI10: now also TP755.1
- net NI11: now also TP756.1
- net NI12: now also TP757.1
- net NI13: now also TP758.1
- net NI14: now also TP759.1
- net NI15: now also TP760.1
- net NI16: now also TP761.1
- net NI17: now also TP762.1
- net NI18: now also TP763.1
- net NI19: now also TP764.1
- net NI2: now also TP747.1
- net NI20: now also TP765.1
- net NI21: now also TP766.1
- net NI22: now also TP767.1
- net NI23: now also TP768.1
- net NI3: now also TP748.1
- net NI4: now also TP749.1
- net NI5: now also TP750.1
- net NI6: now also TP751.1
- net NI7: now also TP752.1
- net NI8: now also TP753.1
- net NI9: now also TP754.1
- net SI0: now also TP713.1
- net SI1: now also TP714.1
- net SI10: now also TP723.1
- net SI11: now also TP724.1
- net SI12: now also TP725.1
- net SI13: now also TP726.1
- net SI14: now also TP727.1
- net SI15: now also TP728.1
- net SI16: now also TP729.1
- net SI17: now also TP730.1
- net SI18: now also TP731.1
- net SI19: now also TP732.1
- net SI2: now also TP715.1
- net SI20: now also TP733.1
- net SI21: now also TP734.1
- net SI22: now also TP735.1
- net SI23: now also TP736.1
- net SI3: now also TP716.1
- net SI4: now also TP717.1
- net SI5: now also TP718.1
- net SI6: now also TP719.1
- net SI7: now also TP720.1
- net SI8: now also TP721.1
- net SI9: now also TP722.1
- net TERM_EN: now also TP678.1
- net U21_BI1: now also TP792.1
- net U21_BI11: now also TP1101.1
- net U21_BI12: now also TP1102.1
- net U21_BI3: now also TP793.1
- net U21_BI4: now also TP794.1
- net U21_BI5: now also TP795.1
- net U21_BI6: now also TP796.1
- net U21_VBB_BI: now also TP778.1
- net U22_BI10: now also TP686.1
- net U22_BI11: now also TP705.1
- net U22_BI12: now also TP684.1
- net U22_BI7: now also TP682.1
- net U22_BI8: now also TP685.1
- net U22_BI9: now also TP687.1
- net U22_VBB_BI: now also TP701.1
- net ~{TERM_EN}: now also TP681.1
- net at Q9.2 (E), Q9.4 (E), R483.1: now also TP689.1
- net at Q12.3 (B), R507.1: now also TP688.1
- net at R260.1, R261.1, R262.1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: now also TP799.1
- net at Q3.2 (E), Q3.4 (E), R265.1: now also TP790.1
- net at Q3.3 (B), R267.1: now also TP789.1
- net at Q1.1 (B), R479.2: now also TP679.1
- net at Q12.2 (E), Q12.4 (E), R508.1: now also TP683.1
- net at Q7.2 (E), Q7.4 (E), R465.1: now also TP791.1

Commit message: tweaks and some schematic notes
Other:
- note added: "2.03V"
- note added: "2.7V / 1.7V / 0V"
- note added: "2.7V / 1V"
- note added: "BI1-BI12 SIGNALS SEEM TO FLOAT AT 1.6V, BUT CAN BE DRIVEN TO 0V OR 2.7V. MAY USE BOTH COMMON MODE AND DIFF MODE SIGNALING"
- note added: "SI/NI SIGNAL LOGIC LEVELS ARE 1.5V/0V"
Changed lines of the file:
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@@
+		)
+	)
+	(text "BI1-BI12 SIGNALS SEEM TO FLOAT\nAT 1.6V, BUT CAN BE DRIVEN TO 0V\nOR 2.7V.\nMAY USE BOTH COMMON MODE AND DIFF\nMODE SIGNALING"
+		(exclude_from_sim no)
+		(at 227.838 122.428 0)
+		(effects
+			(font
+				(size 1.27 1.27)
+			)
 		)
 	)
@@
 		)
 	)
-	(text "2 volts"
+	(text "2.03V"
 		(exclude_from_sim no)
 		(at 303.276 123.19 0)
@@
 		(exclude_from_sim no)
 		(at 440.69 109.728 0)
+		(effects
+			(font
+				(size 1.27 1.27)
+			)
+		)
+	)
+	(text "2.7V / 1.7V / 0V"
+		(exclude_from_sim no)
+		(at 236.22 106.934 0)
 		(effects
 			(font
@@
 		)
 	)
+	(text "2.7V / 1V"
+		(exclude_from_sim no)
+		(at 227.33 113.03 0)
+		(effects
+			(font
+				(size 1.27 1.27)
+			)
+		)
+	)
 	(text "U22 U26"
 		(exclude_from_sim no)
@@
 		(effects
 			(font
+				(size 1.27 1.27)
+			)
+		)
+	)
+	(text "SI/NI SIGNAL LOGIC LEVELS\nARE 1.5V/0V"
+		(exclude_from_sim no)
+		(at 116.332 174.244 0)
+		(effects
+			(font
