File: Pod1.kicad_sch (KiCad schematic)
At the start: 155 parts, among them U69 1NB4-5036 Comparator, U70 1NB4-5036 Comparator

Commit message: Add component values, some more nets
Parts:
- C104, C106: value 10pF -> 2.2pF
- C105, C111, C112, C113, C114, C116, C117, C118, C119, C123, C124, C138, C139, C140, C141, C142, C143, C147, C148, C149, C150, C3, C71: value 330pF -> 360pF
- C155: value ? -> 0.047uF
- R4: footprint Resistor_SMD:R_0603_1608Metric -> hp16717:HP_0603
Changed lines of the file:
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@@
 			)
 		)
-		(property "Value" "330pF"
+		(property "Value" "360pF"
 			(at 483.87 41.9162 0)
 			(effects
@@
 			)
 		)
-		(property "Value" "330pF"
+		(property "Value" "360pF"
 			(at 88.8937 265.43 90)
 			(effects
@@
 			)
 		)
-		(property "Value" "330pF"
+		(property "Value" "360pF"
 			(at 212.09 50.8062 0)
 			(effects
@@
 			)
 		)
-		(property "Value" "330pF"
+		(property "Value" "360pF"
 			(at 406.4 132.0862 0)
 			(effects
@@
 			)
 		)
-		(property "Value" "10pF"
+		(property "Value" "2.2pF"
 			(at 122.682 259.08 0)
 			(effects
@@
 			)
 		)
-		(property "Value" "330pF"
+		(property "Value" "360pF"
 			(at 127 132.0862 0)
 			(effects
@@
 			)
 		)
-		(property "Value" "330pF"
+		(property "Value" "360pF"
 			(at 179.07 148.5962 0)
 			(effects
@@
 			)
 		)
-		(property "Value" "330pF"
+		(property "Value" "360pF"
 			(at 168.91 148.5962 0)
 			(effects
@@
 			)
 		)
-		(property "Value" "330pF"
+		(property "Value" "360pF"
 			(at 200.406 148.336 0)
 			(effects
@@
 			)
 		)
-		(property "Value" "330pF"
+		(property "Value" "360pF"
 			(at 468.376 148.336 0)
 			(effects
@@
 			)
 		)
-		(property "Value" "330pF"
+		(property "Value" "360pF"
 			(at 499.11 41.9162 0)
 			(effects
@@
 			)
 		)
-		(property "Value" "330pF"
+		(property "Value" "360pF"
 			(at 447.04 148.5962 0)
 			(effects
@@
 			)
 		)
-		(property "Value" "330pF"
+		(property "Value" "360pF"
 			(at 227.33 50.8062 0)
 			(effects
@@
 			)
 		)
-		(property "Value" "330pF"
+		(property "Value" "360pF"
 			(at 458.724 148.844 0)
 			(effects
@@
 			)
 		)
-		(property "Value" "330pF"
+		(property "Value" "360pF"
 			(at 165.1 50.8062 0)
 			(effects
@@
 			)
 		)
-		(property "Value" "330pF"
+		(property "Value" "360pF"
 			(at 491.49 41.9162 0)
 			(effects
@@
 			)
 		)
-		(property "Value" "330pF"
+		(property "Value" "360pF"
 			(at 436.88 41.9162 0)
 			(effects
@@
 			)
 		)
-		(property "Value" "330pF"
+		(property "Value" "360pF"
 			(at 219.71 50.8062 0)
 			(effects
@@
 			)
 		)
-		(property "Value" "330pF"
+		(property "Value" "360pF"
 			(at 436.88 148.5962 0)
 			(effects
@@
 			)
 		)
-		(property "Value" "10pF"
+		(property "Value" "2.2pF"
 			(at 122.428 286.512 0)
 			(effects
@@
 			)
 		)
-		(property "Value" "330pF"
+		(property "Value" "360pF"
 			(at 204.47 50.8062 0)
 			(effects
@@
 			)
 		)
-		(property "Value" "330pF"
+		(property "Value" "360pF"
 			(at 190.754 148.844 0)
 			(effects
@@
 			)
 		)
-		(property "Value" "330pF"
+		(property "Value" "360pF"
 			(at 445.77 41.9162 0)
 			(effects
@@
 			)
 		)
-		(property "Value" "?"
+		(property "Value" "0.047uF"
 			(at 467.106 179.324 0)
 			(effects
@@
 			)
 		)
-		(property "Footprint" "Resistor_SMD:R_0603_1608Metric"
+		(property "Footprint" "hp16717:HP_0603"
 			(at 92.71 77.47 0)
 			(effects
@@
 			)
 		)
-		(property "Value" "330pF"
+		(property "Value" "360pF"
 			(at 173.99 50.8062 0)
 			(effects
@@
 			)
 		)
-		(property "Value" "330pF"
+		(property "Value" "360pF"
 			(at 476.25 41.9162 0)
 			(effects

Commit message: complete outer layers
Connections:
- net AP1_CLK renamed AP1_CLK_P
- net TZP1_CLK renamed TZP1_CLK_P
- net ~{AP1_CLK} renamed AP1_CLK_N
- net ~{TZP1_CLK} renamed TZP1_CLK_N
Changed lines of the file:
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@@
 		)
 	)
-	(label "TZP1_CLK"
+	(label "TZP1_CLK_P"
 		(at 534.67 80.01 180)
 		(effects
@@
 		)
 	)
-	(label "~{TZP1_CLK}"
+	(label "TZP1_CLK_N"
 		(at 534.67 92.71 180)
 		(effects
@@
 		)
 	)
-	(label "AP1_CLK"
+	(label "AP1_CLK_P"
 		(at 534.67 74.93 180)
 		(effects
@@
 		)
 	)
-	(label "~{AP1_CLK}"
+	(label "AP1_CLK_N"
 		(at 534.67 87.63 180)
 		(effects
@@
 		)
 	)
-	(hierarchical_label "TZP1_CLK"
+	(hierarchical_label "TZP1_CLK_P"
 		(shape output)
 		(at 547.37 80.01 0)
@@
 		)
 	)
-	(hierarchical_label "~{TZP1_CLK}"
+	(hierarchical_label "TZP1_CLK_N"
 		(shape output)
 		(at 547.37 92.71 0)
@@
 		)
 	)
-	(hierarchical_label "~{AP1_CLK}"
+	(hierarchical_label "AP1_CLK_N"
 		(shape output)
 		(at 547.37 87.63 0)
@@
 		)
 	)
-	(hierarchical_label "AP1_CLK"
+	(hierarchical_label "AP1_CLK_P"
 		(shape output)
 		(at 547.37 74.93 0)

Commit message: add test points
Parts:
- added TP1000: CMP1P, hp16717:HP_TP30, symbol Connector:TestPoint_Alt
- added TP1001, TP1002, TP1013, TP1014: GND, hp16717:HP_TP30, symbol Connector:TestPoint_Alt
- added TP1003: POD1_2_TEST, hp16717:HP_TP30, symbol Connector:TestPoint_Alt
- added TP1005, TP997: CMP9, hp16717:HP_TP30, symbol Connector:TestPoint_Alt
- added TP1006, TP992: -5V2, hp16717:HP_TP30, symbol Connector:TestPoint_Alt
- added TP1007, TP1015: +3V3, hp16717:HP_TP30, symbol Connector:TestPoint_Alt
- added TP1008, TP991, TP993: ?, hp16717:HP_TP30, symbol Connector:TestPoint_Alt
- added TP1009: CMP7, hp16717:HP_TP30, symbol Connector:TestPoint_Alt
- added TP1010, TP998: CMP8, hp16717:HP_TP30, symbol Connector:TestPoint_Alt
- added TP1011: CMP3, hp16717:HP_TP30, symbol Connector:TestPoint_Alt
- added TP1012: CMP2, hp16717:HP_TP30, symbol Connector:TestPoint_Alt
- added TP1016: -3V3, hp16717:HP_TP30, symbol Connector:TestPoint_Alt
- added TP960: POD1A_VREF, hp16717:HP_TP30, symbol Connector:TestPoint_Alt
- added TP965: POD1B_VREF, hp16717:HP_TP30, symbol Connector:TestPoint_Alt
- added TP983: POD1A_TZVREF, hp16717:HP_TP30, symbol Connector:TestPoint_Alt
- added TP984: POD1B_TZVREF, hp16717:HP_TP30, symbol Connector:TestPoint_Alt
- added TP999: CMP1N, hp16717:HP_TP30, symbol Connector:TestPoint_Alt
Connections:
- net +3V3: now also TP1007.1, TP1015.1
- net -3V3: now also TP1016.1
- net -5V2: now also TP1006.1, TP992.1
- net GND: now also TP1001.1, TP1002.1, TP1013.1, TP1014.1
- net POD1A_TZVREF: now also TP983.1
- net POD1A_VREF: now also TP960.1
- net POD1B_TZVREF: now also TP984.1
- net POD1B_VREF: now also TP965.1
- net POD1_2_TEST_SIG: now also TP1003.1
- net at R329.7, U70.27 (CMP_OUT9): now also TP1005.1
- net at R335.7, U70.10 (CMP_OUT2): now also TP1012.1
- net at R335.5, U70.12 (CMP_OUT3): now also TP1011.1
- net at R334.3, U70.23 (CMP_OUT7): now also TP1009.1
- net at R334.1, U70.25 (CMP_OUT8): now also TP1010.1
- net at R146.1, R328.16: now also TP993.1
- net at R328.3, U69.27 (CMP_OUT9): now also TP997.1
- net at R161.1, R334.10: now also TP1008.1
- net at R328.1, U69.19 (2V1?): now also TP991.1
- net at R328.5, U69.25 (CMP_OUT8): now also TP998.1
- net at R329.5, U69.7 (CMP_OUT1): now also TP1000.1
- net at R329.3, U69.8 (CMP_OUT1): now also TP999.1
Other:
- moved on the sheet: C155

Commit message: tweaks and some schematic notes
Other:
- note added: "1.3V"
- note added: "2.15V"
- note added: "2.23V"
- note added: "SWING IS 1.7V TO 2.5V (ACQ ASIC) SWING IS 1V TO 1.7V (TIMING ZOOM)"
- note added: "cmpTest: +10V RAMP TO -10V IN 25us."
- note added: "cmpTest: BURSTS 24.7MHz (-1.8V to -1.1V) 50MHz (-2V to -0.8V)"
- note removed: "to acq chip"
Changed lines of the file:
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@@
 	(generator_version "9.0")
 	(paper "A2")
+	(text "cmpTest:\n+10V RAMP TO -10V IN 25us."
+		(exclude_from_sim no)
+		(at 62.992 56.388 0)
+		(effects
+			(font
+				(size 1.27 1.27)
+			)
+		)
+	)
+	(text "2.23V"
+		(exclude_from_sim no)
+		(at 285.75 55.88 0)
+		(effects
+			(font
+				(size 1.27 1.27)
+			)
+		)
+	)
+	(text "2.15V"
+		(exclude_from_sim no)
+		(at 211.074 60.198 0)
+		(effects
+			(font
+				(size 1.27 1.27)
+			)
+		)
+	)
+	(text "cmpTest: BURSTS\n24.7MHz (-1.8V to -1.1V)\n50MHz (-2V to -0.8V)"
+		(exclude_from_sim no)
+		(at 49.53 264.414 0)
+		(effects
+			(font
+				(size 1.27 1.27)
+			)
+		)
+	)
 	(text "to U21 pin Y25"
 		(exclude_from_sim no)
@@
 		)
 	)
+	(text "1.3V"
+		(exclude_from_sim no)
+		(at 282.956 68.58 0)
+		(effects
+			(font
+				(size 1.27 1.27)
+			)
+		)
+	)
 	(text "POD 1"
 		(exclude_from_sim no)
@@
 		)
 	)
-	(text "to acq chip"
+	(text "2.15V"
+		(exclude_from_sim no)
+		(at 264.414 56.134 0)
+		(effects
+			(font
+				(size 1.27 1.27)
+			)
+		)
+	)
+	(text "SWING IS 1.7V TO 2.5V (ACQ ASIC)\nSWING IS 1V TO 1.7V (TIMING ZOOM)"
 		(exclude_from_sim no)
-		(at 278.384 78.486 0)
+		(at 297.942 94.488 0)
 		(effects
 			(font
@@
 		)
 		(property "Value" "?"
-			(at 267.716 45.974 90)
+			(at 267.716 51.816 0)
 			(effects
 				(font
