File: hp16717.kicad_sch (KiCad schematic)
At the start: 64 parts, among them J1 POD1_2, J2 POD3_4, J3 Conn_02x10_Odd_Even, J4 Conn_02x10_Odd_Even, J5 Conn_02x10_Odd_Even, J6 Conn_02x10_Odd_Even, J7 Conn_02x10_Odd_Even, J8 Conn_02x10_Odd_Even

Commit message: Add component values, some more nets
Parts:
- added C545, C547: 3.3nF, hp16717:HP_0603, symbol Device:C_Small
- added C546: 560pF, hp16717:HP_0805, symbol Device:C_Small
- C110, C152, C153, C216, C228, C242, C243, C244: value ? -> 0.047uF
- C217, C218, C219, C220, C221, C222, C223, C224, C225, C226, C227: value ? -> 3.3nF
Connections:
- net GND: now also C545.1, C546.1, C547.1
Other:
- added sheet Acq RAM 2 (AcqRAM2.kicad_sch)
- sheet Acq RAM 1 ports: added U25_[15..0], U27_[15..0], U29_[15..0], U35_[15..0], U37_[15..0], U46_[15..0], U48_[15..0], U54_[15..0], U56_[15..0]; removed U39_QSF, ~{RAS3}, ~{RAS4}
- sheet Acquisition ASICs ports: added IDB[15..0], POD1A_VREF, POD1B_VREF, POD2A_VREF, POD2B_VREF, POD3A_VREF, POD3B_VREF, POD4A_VREF, POD4B_VREF, U25_[15..0], U27_[15..0], U29_[15..0], U30_[15..0], U32_[15..0], U35_[15..0], U37_[15..0], U39_[15..0], U40_[15..0], U42_[15..0], U46_[15..0], U48_[15..0], U50_[15..0], U52_[15..0], U54_[15..0], U56_[15..0], U58_[15..0], U60_[15..0]; removed none

Commit message: complete outer layers
Parts:
- added H1, H2, H3: MountingHole, hp16717:HP_TOOLING_125, symbol Mechanical:MountingHole
- added MH1, MH2, MH3, MH4: TestPoint, hp16717:HP_PEM_M3, symbol Connector:TestPoint
- C154: value 0.47uF -> 4.7uF; footprint Capacitor_Tantalum_SMD:CP_EIA-3528-21_Kemet-B -> hp16717:HP_CP_EIA-3528
- C159: footprint Capacitor_Tantalum_SMD:CP_EIA-7343-31_Kemet-D -> hp16717:HP_CP_EIA-7343
- FB1, FB2: footprint Inductor_SMD:L_TDK_NLV32_3.2x2.5mm -> hp16717:HP_L_3.2x2.5mm
- S1, S2: footprint Package_SO:SO-8_3.9x4.9mm_P1.27mm -> hp16717:HP_SO-8_3.9x4.9mm_P1.27mm
- TP1, TP2, TP3, TP4, TP5, TP6, TP7: footprint TestPoint:TestPoint_THTPad_D1.0mm_Drill0.5mm -> hp16717:HP_TP_THTPad_D64_Drill48
Connections:
- net GND: now also MH1.1, MH2.1, MH3.1, MH4.1
- net Clocks/TZCLK1 renamed Clocks/TZCLK1_P
- net Clocks/TZCLK2 renamed Clocks/TZCLK2_P
- net Clocks/TZCLK3 renamed Clocks/TZCLK3_P
- net Clocks/TZCLK4 renamed Clocks/TZCLK4_P
- net Clocks/TZCLK5 renamed Clocks/TZCLK5_P
- net Clocks/TZCLKI renamed Clocks/TZCLKI_P
- net Clocks/~{TZCLK1} renamed Clocks/TZCLK1_N
- net Clocks/~{TZCLK2} renamed Clocks/TZCLK2_N
- net Clocks/~{TZCLK3} renamed Clocks/TZCLK3_N
- net Clocks/~{TZCLK4} renamed Clocks/TZCLK4_N
- net Clocks/~{TZCLK5} renamed Clocks/TZCLK5_N
- net Clocks/~{TZCLKI} renamed Clocks/TZCLKI_N
Other:
- sheet Acq RAM 1 ports: added VSC[8..0]; removed none
- sheet Acq RAM 2 ports: added VSC[18..9]; removed none
- sheet Acquisition ASICs ports: added AP1_CLK_N, AP1_CLK_P, AP2_CLK_N, AP2_CLK_P, AP3_CLK_N, AP3_CLK_P, AP4_CLK_N, AP4_CLK_P, FA_UNK1, FPGA_ASIC_XC1, FPGA_ASIC_XC2, IDB_CLK, U21_FPGA[7..0], U21_SYSCLK_N, U21_SYSCLK_P, U22_FPGA[7..0], U22_SYSCLK_N, U22_SYSCLK_P, VSC[18..9], VSC[8..0]; removed AP1_CLK, AP2_CLK, AP3_CLK, AP4_CLK, ~{AP1_CLK}, ~{AP2_CLK}, ~{AP3_CLK}, ~{AP4_CLK}
- sheet Backplane ports: added 100M_SYSCLK2_N, 100M_SYSCLK2_P, FA_UNK1, FPGA_ASIC_XC1, FPGA_ASIC_XC2, IDB_CLK, U21_FPGA[7..0], U21_SYSCLK_N, U21_SYSCLK_P, U22_FPGA[7..0], U22_SYSCLK_N, U22_SYSCLK_P, ~{DAC_WR}; removed 100M_SYSCLK2, ~{100M_SYSCLK2}
- sheet Clocks ports: added 100M_SYSCLK2_N, 100M_SYSCLK2_P, TZCLK1_N, TZCLK1_P, TZCLK2_N, TZCLK2_P, TZCLK3_N, TZCLK3_P, TZCLK4_N, TZCLK4_P, TZCLK5_N, TZCLK5_P, TZCLKI_N, TZCLKI_P, TZCLKO10_N, TZCLKO10_P, TZCLKO1_N, TZCLKO1_P, TZCLKO2_N, TZCLKO2_P, TZCLKO3_N, TZCLKO3_P, TZCLKO4_N, TZCLKO4_P, TZCLKO5_N, TZCLKO5_P, TZCLKO6_N, TZCLKO6_P, TZCLKO7_N, TZCLKO7_P, TZCLKO8_N, TZCLKO8_P, TZCLKO9_N, TZCLKO9_P; removed 100M_SYSCLK2, TZCLK1, TZCLK2, TZCLK3, TZCLK4, TZCLK5, TZCLKI, TZCLKO1, TZCLKO10, TZCLKO2, TZCLKO3, TZCLKO4, TZCLKO5, TZCLKO6, TZCLKO7, TZCLKO8, TZCLKO9, ~{100M_SYSCLK2}, ~{TZCLK1}, ~{TZCLK2}, ~{TZCLK3}, ~{TZCLK4}, ~{TZCLK5}, ~{TZCLKI}, ~{TZCLKO10}, ~{TZCLKO1}, ~{TZCLKO2}, ~{TZCLKO3}, ~{TZCLKO4}, ~{TZCLKO5}, ~{TZCLKO6}, ~{TZCLKO7}, ~{TZCLKO8}, ~{TZCLKO9}
- sheet Pod 1 Comparator ports: added AP1_CLK_N, AP1_CLK_P, TZP1_CLK_N, TZP1_CLK_P; removed AP1_CLK, TZP1_CLK, ~{AP1_CLK}, ~{TZP1_CLK}
- sheet Pod 2 Comparator ports: added AP2_CLK_N, AP2_CLK_P, TZP2_CLK_N, TZP2_CLK_P; removed AP2_CLK, TZP2_CLK, ~{AP2_CLK}, ~{TZP2_CLK}
- sheet Pod 3 Comparator ports: added AP3_CLK_N, AP3_CLK_P, TZP3_CLK_N, TZP3_CLK_P; removed AP3_CLK, TZP3_CLK, ~{AP3_CLK}, ~{TZP3_CLK}
- sheet Pod 4 Comparator ports: added AP4_CLK_N, AP4_CLK_P, TZP4_CLK_N, TZP4_CLK_P; removed AP4_CLK, TZP4_CLK, ~{AP4_CLK}, ~{TZP4_CLK}
- sheet TimingZoom ports: added TZCLKO10_N, TZCLKO10_P, TZCLKO1_N, TZCLKO1_P, TZCLKO2_N, TZCLKO2_P, TZCLKO3_N, TZCLKO3_P, TZCLKO4_N, TZCLKO4_P, TZCLKO5_N, TZCLKO5_P, TZCLKO6_N, TZCLKO6_P, TZCLKO7_N, TZCLKO7_P, TZCLKO8_N, TZCLKO8_P, TZCLKO9_N, TZCLKO9_P, TZP1_CLK_N, TZP1_CLK_P, TZP2_CLK_N, TZP2_CLK_P, TZP3_CLK_N, TZP3_CLK_P, TZP4_CLK_N, TZP4_CLK_P; removed TZCLKO1, TZCLKO10, TZCLKO2, TZCLKO3, TZCLKO4, TZCLKO5, TZCLKO6, TZCLKO7, TZCLKO8, TZCLKO9, TZP1_CLK, TZP2_CLK, TZP3_CLK, TZP4_CLK, ~{TZCLKO10}, ~{TZCLKO1}, ~{TZCLKO2}, ~{TZCLKO3}, ~{TZCLKO4}, ~{TZCLKO5}, ~{TZCLKO6}, ~{TZCLKO7}, ~{TZCLKO8}, ~{TZCLKO9}, ~{TZP1_CLK}, ~{TZP2_CLK}, ~{TZP3_CLK}, ~{TZP4_CLK}
- note added: "PEM FASTENERS"
- note added: "TOOLING HOLES"

Commit message: schematic cleanup, arrange silk designators
Connections:
- net +3V3: now also C545.2, C546.2, C547.2
Other:
- sheet Acquisition ASICs ports: added U21_VBB_BI, U22_VBB_BI; removed none
- sheet Clocks ports: added none; removed TZCLK6, TZCLK7, ~{TZCLK6}, ~{TZCLK7}
- sheet HS Interconnect ports: added U21_VBB_BI, U22_VBB_BI; removed none
- moved on the sheet: C216, C217, C218, C219, C220, C221, C222, C223, C224, C225, C228, C545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

Commit message: numerous small fixes, add plane and inner signal layers
Connections:
- net Clocks/TZCLK1_N renamed TZCLK1_N
- net Clocks/TZCLK1_P renamed TZCLK1_P
- net Clocks/TZCLK2_N renamed TZCLK2_N
- net Clocks/TZCLK2_P renamed TZCLK2_P
- net Clocks/TZCLK3_N renamed TZCLK3_N
- net Clocks/TZCLK3_P renamed TZCLK3_P
- net Clocks/TZCLK4_N renamed TZCLK4_N
- net Clocks/TZCLK4_P renamed TZCLK4_P
- net Clocks/TZCLK5_N renamed TZCLK5_N
- net Clocks/TZCLK5_P renamed TZCLK5_P
- net Clocks/TZCLKI_N renamed TZCLKI_N
- net Clocks/TZCLKI_P renamed TZCLKI_P
Changed lines of the file:
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@@
 		)
 	)
+	(wire
+		(pts
+			(xy 120.65 326.39) (xy 129.54 326.39)
+		)
+		(stroke
+			(width 0)
+			(type default)
+		)
+	)
 	(bus
 		(pts
@@
 	(wire
 		(pts
+			(xy 121.92 328.93) (xy 129.54 328.93)
+		)
+		(stroke
+			(width 0)
+			(type default)
+		)
+	)
+	(wire
+		(pts
 			(xy 419.1 262.89) (xy 419.1 265.43)
 		)
@@
 	(wire
 		(pts
-			(xy 120.65 328.93) (xy 120.65 341.63)
+			(xy 120.65 326.39) (xy 120.65 341.63)
 		)
 		(stroke
@@
 	(wire
 		(pts
-			(xy 129.54 326.39) (xy 121.92 326.39)
-		)
-		(stroke
-			(width 0)
-			(type default)
-		)
-	)
-	(wire
-		(pts
 			(xy 57.15 246.38) (xy 57.15 254)
 		)
@@
 	(wire
 		(pts
-			(xy 121.92 326.39) (xy 121.92 339.09)
+			(xy 121.92 328.93) (xy 121.92 339.09)
 		)
 		(stroke
@@
 	(wire
 		(pts
-			(xy 129.54 328.93) (xy 120.65 328.93)
-		)
-		(stroke
-			(width 0)
-			(type default)
-		)
-	)
-	(wire
-		(pts
 			(xy 453.39 231.14) (xy 453.39 229.87)
 		)
@@
 		)
 	)
+	(label "TZCLK1_N"
+		(at 549.91 228.6 90)
+		(effects
+			(font
+				(size 1.27 1.27)
+			)
+			(justify left bottom)
+		)
+	)
 	(label "P1_D14"
 		(at 80.01 125.73 0)
@@
 		)
 	)
+	(label "TZCLKI_P"
+		(at 377.19 229.87 90)
+		(effects
+			(font
+				(size 1.27 1.27)
+			)
+			(justify left bottom)
+		)
+	)
 	(label "P4_D15"
 		(at 48.26 287.02 0)
@@
 		)
 	)
+	(label "TZCLK1_P"
+		(at 563.88 219.71 0)
+		(effects
+			(font
+				(size 1.27 1.27)
+			)
+			(justify left bottom)
+		)
+	)
 	(label "TZCLKO1_P"
 		(at 579.12 129.54 180)
@@
 		)
 	)
+	(label "TZCLK4_N"
+		(at 448.31 229.87 90)
+		(effects
+			(font
+				(size 1.27 1.27)
+			)
+			(justify left bottom)
+		)
+	)
+	(label "TZCLKI_N"
+		(at 401.32 228.6 90)
+		(effects
+			(font
+				(size 1.27 1.27)
+			)
+			(justify left bottom)
+		)
+	)
 	(label "TZCLKO2_P"
 		(at 257.81 257.81 180)
@@
 		)
 	)
+	(label "TZCLK3_N"
+		(at 488.95 228.6 90)
+		(effects
+			(font
+				(size 1.27 1.27)
+			)
+			(justify left bottom)
+		)
+	)
 	(label "TZCLKO9_N"
 		(at 579.12 172.72 180)
@@
 		)
 	)
+	(label "TZCLK3_P"
+		(at 501.65 219.71 0)
+		(effects
+			(font
+				(size 1.27 1.27)
+			)
+			(justify left bottom)
+		)
+	)
 	(label "TZCLKO8_N"
 		(at 257.81 290.83 180)
@@
 		)
 	)
+	(label "TZCLK2_N"
+		(at 516.89 228.6 90)
+		(effects
+			(font
+				(size 1.27 1.27)
+			)
+			(justify left bottom)
+		)
+	)
 	(label "P1_D2"
 		(at 80.01 80.01 0)
@@
 		)
 	)
+	(label "TZCLK5_N"
+		(at 416.56 229.87 90)
+		(effects
+			(font
+				(size 1.27 1.27)
+			)
+			(justify left bottom)
+		)
+	)
 	(label "P2_D10"
 		(at 48.26 110.49 0)
@@
 		)
 	)
+	(label "TZCLK2_P"
+		(at 532.13 219.71 0)
+		(effects
+			(font
+				(size 1.27 1.27)
+			)
+			(justify left bottom)
+		)
+	)
 	(label "P3_CLK"
 		(at 80.01 297.18 0)
@@
 		)
 	)
+	(label "TZCLK4_P"
+		(at 466.09 219.71 0)
+		(effects
+			(font
+				(size 1.27 1.27)
+			)
+			(justify left bottom)
+		)
+	)
 	(label "P4_D12"
 		(at 48.26 274.32 0)
@@
 		(effects
 			(font
+				(size 1.27 1.27)
+			)
+			(justify left bottom)
+		)
+	)
+	(label "TZCLK5_P"
+		(at 433.07 219.71 0)
+		(effects
+			(font

Commit message: add test points
Parts:
- added TP1022, TP1051: +5V, hp16717:HP_TP30, symbol Connector:TestPoint_Alt
- added TP1023, TP1053: GND, hp16717:HP_TP30, symbol Connector:TestPoint_Alt
- added TP1024, TP1050, TP1089, TP1090, TP1091, TP1092, TP1093, TP1094, TP1095, TP1096, TP1097, TP1098, TP1099, TP1100: ?, hp16717:HP_TP30, symbol Connector:TestPoint_Alt
- added TP1052: POD_PWR_EN, hp16717:HP_TP30, symbol Connector:TestPoint_Alt
- added TP1074: TZCLKI_P, hp16717:HP_TP30, symbol Connector:TestPoint_Alt
- added TP1075: TZCLKI_N, hp16717:HP_TP30, symbol Connector:TestPoint_Alt
- added TP1076: TZCLK5_N, hp16717:HP_TP30, symbol Connector:TestPoint_Alt
- added TP1077: TZCLK5_P, hp16717:HP_TP30, symbol Connector:TestPoint_Alt
- added TP1078: TZCLK4_P, hp16717:HP_TP30, symbol Connector:TestPoint_Alt
- added TP1079: TZCLK4_N, hp16717:HP_TP30, symbol Connector:TestPoint_Alt
- added TP1080: TZCLK3_N, hp16717:HP_TP30, symbol Connector:TestPoint_Alt
- added TP1081: TZCLK3_P, hp16717:HP_TP30, symbol Connector:TestPoint_Alt
- added TP1082: TZCLK2_P, hp16717:HP_TP30, symbol Connector:TestPoint_Alt
- added TP1083: TZCLK2_N, hp16717:HP_TP30, symbol Connector:TestPoint_Alt
- added TP1084: TZCLK1_P, hp16717:HP_TP30, symbol Connector:TestPoint_Alt
- added TP1085: TZCLK1_N, hp16717:HP_TP30, symbol Connector:TestPoint_Alt
- added TP1086: MASTERCARD, hp16717:HP_TP30, symbol Connector:TestPoint_Alt
- added TP1087: EXP1, hp16717:HP_TP30, symbol Connector:TestPoint_Alt
- added TP1088: EXP2, hp16717:HP_TP30, symbol Connector:TestPoint_Alt
Connections:
- net +3V3: now also TP1099.1
- net +5V: now also TP1022.1, TP1051.1
- net Backplane/EXT1: now also TP1087.1
- net Backplane/EXT2: now also TP1088.1
- net Backplane/MASTERCARD: now also TP1086.1
- net Backplane/~{POD_PWR_EN}: now also TP1052.1
- net GND: now also TP1023.1, TP1053.1
- net TZCLK1_N: now also TP1085.1
- net TZCLK1_P: now also TP1084.1
- net TZCLK2_N: now also TP1083.1
- net TZCLK2_P: now also TP1082.1
- net TZCLK3_N: now also TP1080.1
- net TZCLK3_P: now also TP1081.1
- net TZCLK4_N: now also TP1079.1
- net TZCLK4_P: now also TP1078.1
- net TZCLK5_N: now also TP1076.1
- net TZCLK5_P: now also TP1077.1
- net TZCLKI_N: now also TP1075.1
- net TZCLKI_P: now also TP1074.1
- net at C243.1, FB2.1, S2.5 (OUT)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: now also TP1050.1
- net at J6.6 (Pin_6), J6.8 (Pin_8), R196.2: now also TP1093.1
- net at C228.2, J6.11 (Pin_11), R258.2: now also TP1100.1
- net at J4.2 (Pin_2), J4.4 (Pin_4), R189.2: now also TP1090.1
- net at J4.6 (Pin_6), J4.8 (Pin_8), R194.2: now also TP1089.1
- net at C110.1, FB1.1, S1.5 (OUT)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: now also TP1024.1
- net at J8.6 (Pin_6), J8.8 (Pin_8), R198.2: now also TP1097.1
- net at J6.2 (Pin_2), J6.4 (Pin_4), R502.2: now also TP1094.1
- net at J8.2 (Pin_2), J8.4 (Pin_4), R193.2: now also TP1098.1
- net at J7.2 (Pin_2), J7.4 (Pin_4), R192.2: now also TP1096.1
- net at J5.6 (Pin_6), J5.8 (Pin_8), R195.2: now also TP1091.1
- net at J5.2 (Pin_2), J5.4 (Pin_4), R506.2: now also TP1092.1
- net at J7.6 (Pin_6), J7.8 (Pin_8), R197.2: now also TP1095.1
Other:
- moved on the sheet: C228

Commit message: tweaks and some schematic notes
Parts:
- removed J3: Conn_02x10_Odd_Even, hp16717:AMP_5-104069-1, symbol Connector_Generic:Conn_02x10_Odd_Even
- added J3: Conn_02x10_Odd_Even_MountingPin, hp16717:AMP_5-104069-1, symbol Connector_Generic_MountingPin:Conn_02x10_Odd_Even_MountingPin
Connections:
- net Backplane/EXT1: now also J3.12 (Pin_12)
- net Backplane/EXT2: now also J3.10 (Pin_10)
- net Backplane/MASTERCARD: now also J3.11 (Pin_11)
- net GND: now also J3.1 (Pin_1), J3.13 (Pin_13), J3.14 (Pin_14), J3.15 (Pin_15), J3.18 (Pin_18), J3.19 (Pin_19), J3.20 (Pin_20), J3.3 (Pin_3), J3.5 (Pin_5), J3.7 (Pin_7), J3.9 (Pin_9), J3.MP (MountPin)
- net Pod 1 Comparator/POD1_2_TEST_SIG: now also J3.6 (Pin_6), J3.8 (Pin_8)
- net Pod 3 Comparator/POD3_4_TEST_SIG: now also J3.2 (Pin_2), J3.4 (Pin_4)
- net TZCLKI_N: now also J3.16 (Pin_16)
- net TZCLKI_P: now also J3.17 (Pin_17)
