File: AcqRAM1.kicad_sch (KiCad schematic)
At the start: 74 parts, among them U25 MSM5416283, U26 MSM5416283, U27 MSM5416283, U28 MSM5416283, U29 MSM5416283, U30 MSM5416283, U31 MSM5416283, U32 MSM5416283, U33 MSM5416283, U35 MSM5416283, U36 MSM5416283, U37 MSM5416283, U38 MSM5416283, U39 MSM5416283, U40 MSM5416283, U41 MSM5416283, U42 MSM5416283, U43 MSM5416283, U46 MSM5416283, U47 MSM5416283, U48 MSM5416283, U49 MSM5416283, U50 MSM5416283, U51 MSM5416283, U52 MSM5416283, U53 MSM5416283, U54 MSM5416283, U55 MSM5416283, U56 MSM5416283, U57 MSM5416283, U58 MSM5416283, U59 MSM5416283, U60 MSM5416283, U61 MSM5416283

Commit message: Add component values, some more nets
Parts:
- removed U30, U31, U32, U33, U39, U40, U41, U42, U43, U50, U51, U52, U53, U58, U59, U60, U61: MSM5416283, hp16717:HP_SOIC-64, symbol hp16717:MSM5416283
- C489, C490, C492, C493, C495, C497, C498, C499, C500, C501, C502, C503, C504, C505, C506, C507, C508, C509, C512, C513, C514, C515, C516, C517, C518, C519, C520: value ? -> 0.047uF
- C491, C494, C496, C510, C511: value ? -> 360pF
Connections:
- net U56_3: now reaches U57.11 (SDQ3)
- net U56_3: now also U56.11 (SDQ3)
- net U56_4: now reaches U57.14 (SDQ4)
- net U56_4: now also U56.14 (SDQ4)
- net U56_5: now reaches U57.16 (SDQ5)
- net U56_5: now also U56.16 (SDQ5)
- net U56_6: now reaches U57.19 (SDQ6)
- net U56_6: now also U56.19 (SDQ6)
- net U56_7: now reaches U57.21 (SDQ7)
- net U56_7: now also U56.21 (SDQ7)
- net U56_0: now reaches U57.4 (SDQ0)
- net U56_0: now also U56.4 (SDQ0)
- net U56_8: now reaches U57.44 (SDQ8)
- net U56_8: now also U56.44 (SDQ8)
- net U56_9: now reaches U57.46 (SDQ9)
- net U56_9: now also U56.46 (SDQ9)
- net U56_10: now reaches U57.49 (SDQ10)
- net U56_10: now also U56.49 (SDQ10)
- net U56_11: now reaches U57.51 (SDQ11)
- net U56_11: now also U56.51 (SDQ11)
- net U56_12: now reaches U57.54 (SDQ12)
- net U56_12: now also U56.54 (SDQ12)
- net U56_13: now reaches U57.56 (SDQ13)
- net U56_13: now also U56.56 (SDQ13)
- net U56_14: now reaches U57.59 (SDQ14)
- net U56_14: now also U56.59 (SDQ14)
- net U56_1: now reaches U57.6 (SDQ1)
- net U56_1: now also U56.6 (SDQ1)
- net U56_15: now reaches U57.61 (SDQ15)
- net U56_15: now also U56.61 (SDQ15)
- net U56_2: now reaches U57.9 (SDQ2)
- net U56_2: now also U56.9 (SDQ2)
- net U46_3: now reaches U46.11 (SDQ3)
- net U46_3: now also U47.11 (SDQ3)
- net U46_4: now reaches U46.14 (SDQ4)
- net U46_4: now also U47.14 (SDQ4)
- net U46_5: now reaches U46.16 (SDQ5)
- net U46_5: now also U47.16 (SDQ5)
- net U46_6: now reaches U46.19 (SDQ6)
- net U46_6: now also U47.19 (SDQ6)
- net U46_7: now reaches U46.21 (SDQ7)
- net U46_7: now also U47.21 (SDQ7)
- net U46_0: now reaches U46.4 (SDQ0)
- net U46_0: now also U47.4 (SDQ0)
- net U46_8: now reaches U46.44 (SDQ8)
- net U46_8: now also U47.44 (SDQ8)
- net U46_9: now reaches U46.46 (SDQ9)
- net U46_9: now also U47.46 (SDQ9)
- net U46_10: now reaches U46.49 (SDQ10)
- net U46_10: now also U47.49 (SDQ10)
- net U46_11: now reaches U46.51 (SDQ11)
- net U46_11: now also U47.51 (SDQ11)
- net U46_12: now reaches U46.54 (SDQ12)
- net U46_12: now also U47.54 (SDQ12)
- net U46_13: now reaches U46.56 (SDQ13)
- net U46_13: now also U47.56 (SDQ13)
- net U46_14: now reaches U46.59 (SDQ14)
- net U46_14: now also U47.59 (SDQ14)
- net U46_1: now reaches U46.6 (SDQ1)
- net U46_1: now also U47.6 (SDQ1)
- net U46_15: now reaches U46.61 (SDQ15)
- net U46_15: now also U47.61 (SDQ15)
- net U46_2: now reaches U46.9 (SDQ2)
- net U46_2: now also U47.9 (SDQ2)
- net U54_3: now reaches U55.11 (SDQ3)
- net U54_3: now also U54.11 (SDQ3)
- net U54_4: now reaches U55.14 (SDQ4)
- net U54_4: now also U54.14 (SDQ4)
- net U54_5: now reaches U55.16 (SDQ5)
- net U54_5: now also U54.16 (SDQ5)
- net U54_6: now reaches U55.19 (SDQ6)
- net U54_6: now also U54.19 (SDQ6)
- net U54_7: now reaches U55.21 (SDQ7)
- net U54_7: now also U54.21 (SDQ7)
- net U54_0: now reaches U55.4 (SDQ0)
- net U54_0: now also U54.4 (SDQ0)
- net U54_8: now reaches U55.44 (SDQ8)
- net U54_8: now also U54.44 (SDQ8)
- net U54_9: now reaches U55.46 (SDQ9)
- net U54_9: now also U54.46 (SDQ9)
- net U54_10: now reaches U55.49 (SDQ10)
- net U54_10: now also U54.49 (SDQ10)
- net U54_11: now reaches U55.51 (SDQ11)
- net U54_11: now also U54.51 (SDQ11)
- net U54_12: now reaches U55.54 (SDQ12)
- net U54_12: now also U54.54 (SDQ12)
- net U54_13: now reaches U55.56 (SDQ13)
- net U54_13: now also U54.56 (SDQ13)
- net U54_14: now reaches U55.59 (SDQ14)
- net U54_14: now also U54.59 (SDQ14)
- net U54_1: now reaches U55.6 (SDQ1)
- net U54_1: now also U54.6 (SDQ1)
- net U54_15: now reaches U55.61 (SDQ15)
- net U54_15: now also U54.61 (SDQ15)
- net U54_2: now reaches U55.9 (SDQ2)
- net U54_2: now also U54.9 (SDQ2)
- net U29_3: now reaches U29.11 (SDQ3)
- net U29_4: now reaches U29.14 (SDQ4)
- net U29_5: now reaches U29.16 (SDQ5)
- net U29_6: now reaches U29.19 (SDQ6)
- net U29_7: now reaches U29.21 (SDQ7)
- net U29_0: now reaches U29.4 (SDQ0)
- net U29_8: now reaches U29.44 (SDQ8)
- net U29_9: now reaches U29.46 (SDQ9)
- net U29_10: now reaches U29.49 (SDQ10)
- net U29_11: now reaches U29.51 (SDQ11)
- net U29_12: now reaches U29.54 (SDQ12)
- net U29_13: now reaches U29.56 (SDQ13)
- net U29_14: now reaches U29.59 (SDQ14)
- net U29_1: now reaches U29.6 (SDQ1)
- net U29_15: now reaches U29.61 (SDQ15)
- net U29_2: now reaches U29.9 (SDQ2)
- net U37_3: now reaches U37.11 (SDQ3)
- net U37_3: now also U38.11 (SDQ3)
- net U37_4: now reaches U37.14 (SDQ4)
- net U37_4: now also U38.14 (SDQ4)
- net U37_5: now reaches U37.16 (SDQ5)
- net U37_5: now also U38.16 (SDQ5)
- net U37_6: now reaches U37.19 (SDQ6)
- net U37_6: now also U38.19 (SDQ6)
- net U37_7: now reaches U37.21 (SDQ7)
- net U37_7: now also U38.21 (SDQ7)
- net U37_0: now reaches U37.4 (SDQ0)
- net U37_0: now also U38.4 (SDQ0)
- net U37_8: now reaches U37.44 (SDQ8)
- net U37_8: now also U38.44 (SDQ8)
- net U37_9: now reaches U37.46 (SDQ9)
- net U37_9: now also U38.46 (SDQ9)
- net U37_10: now reaches U37.49 (SDQ10)
- net U37_10: now also U38.49 (SDQ10)
- net U37_11: now reaches U37.51 (SDQ11)
- net U37_11: now also U38.51 (SDQ11)
- net U37_12: now reaches U37.54 (SDQ12)
- net U37_12: now also U38.54 (SDQ12)
- net U37_13: now reaches U37.56 (SDQ13)
- net U37_13: now also U38.56 (SDQ13)
- net U37_14: now reaches U37.59 (SDQ14)
- net U37_14: now also U38.59 (SDQ14)
- net U37_1: now reaches U37.6 (SDQ1)
- net U37_1: now also U38.6 (SDQ1)
- net U37_15: now reaches U37.61 (SDQ15)
- net U37_15: now also U38.61 (SDQ15)
- net U37_2: now reaches U37.9 (SDQ2)
- net U37_2: now also U38.9 (SDQ2)
- net U27_3: now reaches U27.11 (SDQ3)
- net U27_3: now also U28.11 (SDQ3)
- net U27_4: now reaches U27.14 (SDQ4)
- net U27_4: now also U28.14 (SDQ4)
- net U27_5: now reaches U27.16 (SDQ5)
- net U27_5: now also U28.16 (SDQ5)
- net U27_6: now reaches U27.19 (SDQ6)
- net U27_6: now also U28.19 (SDQ6)
- net U27_7: now reaches U27.21 (SDQ7)
- net U27_7: now also U28.21 (SDQ7)
- net U27_0: now reaches U27.4 (SDQ0)
- net U27_0: now also U28.4 (SDQ0)
- net U27_8: now reaches U27.44 (SDQ8)
- net U27_8: now also U28.44 (SDQ8)
- net U27_9: now reaches U27.46 (SDQ9)
- net U27_9: now also U28.46 (SDQ9)
- net U27_10: now reaches U27.49 (SDQ10)
- net U27_10: now also U28.49 (SDQ10)
- net U27_11: now reaches U27.51 (SDQ11)
- net U27_11: now also U28.51 (SDQ11)
- net U27_12: now reaches U27.54 (SDQ12)
- net U27_12: now also U28.54 (SDQ12)
- net U27_13: now reaches U27.56 (SDQ13)
- net U27_13: now also U28.56 (SDQ13)
- net U27_14: now reaches U27.59 (SDQ14)
- net U27_14: now also U28.59 (SDQ14)
- net U27_1: now reaches U27.6 (SDQ1)
- net U27_1: now also U28.6 (SDQ1)
- net U27_15: now reaches U27.61 (SDQ15)
- net U27_15: now also U28.61 (SDQ15)
- net U27_2: now reaches U27.9 (SDQ2)
- net U27_2: now also U28.9 (SDQ2)
- net U35_3: now reaches U35.11 (SDQ3)
- net U35_3: now also U36.11 (SDQ3)
- net U35_4: now reaches U35.14 (SDQ4)
- net U35_4: now also U36.14 (SDQ4)
- net U35_5: now reaches U35.16 (SDQ5)
- net U35_5: now also U36.16 (SDQ5)
- net U35_6: now reaches U35.19 (SDQ6)
- net U35_6: now also U36.19 (SDQ6)
- net U35_7: now reaches U35.21 (SDQ7)
- net U35_7: now also U36.21 (SDQ7)
- net U35_0: now reaches U35.4 (SDQ0)
- net U35_0: now also U36.4 (SDQ0)
- net U35_8: now reaches U35.44 (SDQ8)
- net U35_8: now also U36.44 (SDQ8)
- net U35_9: now reaches U35.46 (SDQ9)
- net U35_9: now also U36.46 (SDQ9)
- net U35_10: now reaches U35.49 (SDQ10)
- net U35_10: now also U36.49 (SDQ10)
- net U35_11: now reaches U35.51 (SDQ11)
- net U35_11: now also U36.51 (SDQ11)
- net U35_12: now reaches U35.54 (SDQ12)
- net U35_12: now also U36.54 (SDQ12)
- net U35_13: now reaches U35.56 (SDQ13)
- net U35_13: now also U36.56 (SDQ13)
- net U35_14: now reaches U35.59 (SDQ14)
- net U35_14: now also U36.59 (SDQ14)
- net U35_1: now reaches U35.6 (SDQ1)
- net U35_1: now also U36.6 (SDQ1)
- net U35_15: now reaches U35.61 (SDQ15)
- net U35_15: now also U36.61 (SDQ15)
- net U35_2: now reaches U35.9 (SDQ2)
- net U35_2: now also U36.9 (SDQ2)
- net U25_3: now reaches U25.11 (SDQ3)
- net U25_3: now also U26.11 (SDQ3)
- net U25_4: now reaches U25.14 (SDQ4)
- net U25_4: now also U26.14 (SDQ4)
- net U25_5: now reaches U25.16 (SDQ5)
- net U25_5: now also U26.16 (SDQ5)
- net U25_6: now reaches U25.19 (SDQ6)
- net U25_6: now also U26.19 (SDQ6)
- net U25_7: now reaches U25.21 (SDQ7)
- net U25_7: now also U26.21 (SDQ7)
- net U25_0: now reaches U25.4 (SDQ0)
- net U25_0: now also U26.4 (SDQ0)
- net U25_8: now reaches U25.44 (SDQ8)
- net U25_8: now also U26.44 (SDQ8)
- net U25_9: now reaches U25.46 (SDQ9)
- net U25_9: now also U26.46 (SDQ9)
- net U25_10: now reaches U25.49 (SDQ10)
- net U25_10: now also U26.49 (SDQ10)
- net U25_11: now reaches U25.51 (SDQ11)
- net U25_11: now also U26.51 (SDQ11)
- net U25_12: now reaches U25.54 (SDQ12)
- net U25_12: now also U26.54 (SDQ12)
- net U25_13: now reaches U25.56 (SDQ13)
- net U25_13: now also U26.56 (SDQ13)
- net U25_14: now reaches U25.59 (SDQ14)
- net U25_14: now also U26.59 (SDQ14)
- net U25_1: now reaches U25.6 (SDQ1)
- net U25_1: now also U26.6 (SDQ1)
- net U25_15: now reaches U25.61 (SDQ15)
- net U25_15: now also U26.61 (SDQ15)
- net U25_2: now reaches U25.9 (SDQ2)
- net U25_2: now also U26.9 (SDQ2)
- net U48_3: now reaches U49.11 (SDQ3)
- net U48_3: now also U48.11 (SDQ3)
- net U48_4: now reaches U49.14 (SDQ4)
- net U48_4: now also U48.14 (SDQ4)
- net U48_5: now reaches U49.16 (SDQ5)
- net U48_5: now also U48.16 (SDQ5)
- net U48_6: now reaches U49.19 (SDQ6)
- net U48_6: now also U48.19 (SDQ6)
- net U48_7: now reaches U49.21 (SDQ7)
- net U48_7: now also U48.21 (SDQ7)
- net U48_0: now reaches U49.4 (SDQ0)
- net U48_0: now also U48.4 (SDQ0)
- net U48_8: now reaches U49.44 (SDQ8)
- net U48_8: now also U48.44 (SDQ8)
- net U48_9: now reaches U49.46 (SDQ9)
- net U48_9: now also U48.46 (SDQ9)
- net U48_10: now reaches U49.49 (SDQ10)
- net U48_10: now also U48.49 (SDQ10)
- net U48_11: now reaches U49.51 (SDQ11)
- net U48_11: now also U48.51 (SDQ11)
- net U48_12: now reaches U49.54 (SDQ12)
- net U48_12: now also U48.54 (SDQ12)
- net U48_13: now reaches U49.56 (SDQ13)
- net U48_13: now also U48.56 (SDQ13)
- net U48_14: now reaches U49.59 (SDQ14)
- net U48_14: now also U48.59 (SDQ14)
- net U48_1: now reaches U49.6 (SDQ1)
- net U48_1: now also U48.6 (SDQ1)
- net U48_15: now reaches U49.61 (SDQ15)
- net U48_15: now also U48.61 (SDQ15)
- net U48_2: now reaches U49.9 (SDQ2)
- net U48_2: now also U48.9 (SDQ2)
Other:
- note added: "A6"
- note added: "AA2"
- note added: "AA4"
- note added: "AA5"
- note added: "AB2"
- note added: "AB3"
- note added: "AB4"
- note added: "AB5"
- note added: "AC2"
- note added: "AC3"
- note added: "AC4"
- note added: "AC5"
- note added: "AD1"
- note added: "AD2"
- note added: "AD3"
- note added: "AD4"
- note added: "AD5"
- note added: "AE10"
- note added: "AE11"
- note added: "AE13"
- note added: "AE2"
- note added: "AE3"
- note added: "AE4"
- note added: "AE5"
- note added: "AE6"
- note added: "AE7"
- note added: "AE8"
- note added: "AE9"
- note added: "AF10"
- note added: "AF11"
- note added: "AF12"
- note added: "AF2"
- note added: "AF3"
- note added: "AF4"
- note added: "AF5"
- note added: "AF6"
- note added: "AF7"
- note added: "AF8"
- note added: "AF9"
- note added: "AG10"
- note added: "AG11"
- note added: "AG12"
- note added: "AG2"
- note added: "AG3"
- note added: "AG4"
- note added: "AG5"
- note added: "AG6"
- note added: "AG7"
- note added: "AG8"
- note added: "AG9"
- note added: "AH2"
- note added: "AH3"
- note added: "AJ6"
- note added: "B3"
- note added: "C10"
- note added: "C11"
- note added: "C12"
- note added: "C2"
- note added: "C3"
- note added: "C4"
- note added: "C5"
- note added: "C6"
- note added: "C7"
- note added: "C8"
- note added: "C9"
- note added: "D10"
- note added: "D11"
- note added: "D12"
- note added: "D14"
- note added: "D2"
- note added: "D3"
- note added: "D4"
- note added: "D5"
- note added: "D6"
- note added: "D7"
- note added: "D8"
- note added: "D9"
- note added: "E10"
- note added: "E11"
- note added: "E12"
- note added: "E13"
- note added: "E2"
- note added: "E3"
- note added: "E4"
- note added: "E5"
- note added: "E6"
- note added: "E7"
- note added: "E8"
- note added: "E9"
- note added: "F1"
- note added: "F2"
- note added: "F3"
- note added: "F4"
- note added: "F5"
- note added: "G2"
- note added: "G3"
- note added: "G4"
- note added: "G5"
- note added: "H2"
- note added: "H3"
- note added: "H4"
- note added: "H5"
- note added: "J2"
- note added: "J3"
- note added: "J4"
- note added: "J5"
- note added: "K2"
- note added: "K3"
- note added: "K4"
- note added: "K5"
- note added: "L2"
- note added: "L3"
- note added: "L4"
- note added: "L5"
- note added: "M2"
- note added: "M3"
- note added: "M4"
- note added: "M5"
- note added: "N1"
- note added: "N2"
- note added: "N3"
- note added: "N4"
- note added: "N5"
- note added: "P2"
- note added: "P3"
- note added: "P4"
- note added: "P5"
- note added: "PIN"
- note added: "R2"
- note added: "R3"
- note added: "R4"
- note added: "R5"
- note added: "T2"
- note added: "T3"
- note added: "T4"
- note added: "T5"
- note added: "U1"
- note added: "U2"
- note added: "U3"
- note added: "U4"
- note added: "U5"
- note added: "V2"
- note added: "V3"
- note added: "V4"
- note added: "V5"
- note added: "W2"
- note added: "W3"
- note added: "W4"
- note added: "W5"
- note added: "Y2"
- note added: "Y3"
- note added: "Y4"
- note added: "Y5"
- moved on the sheet: C481, C482, C483, C484, C485, C486, C487, C488, C489, C490, C491, C492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

Commit message: complete outer layers
Parts:
- C481, C482, C483, C484, C485, C486, C487, C488: value 0.47uF -> 4.7uF; footprint Capacitor_Tantalum_SMD:CP_EIA-3528-21_Kemet-B -> hp16717:HP_CP_EIA-3528
Connections:
- net VSC5: now reaches U57.64 (SC)
- net VSC5: now also U49.64 (SC)
- net VSC0: now reaches U46.64 (SC)
- net VSC0: now also U54.64 (SC)
- net VSC1: now reaches U55.64 (SC)
- net VSC1: now also U47.64 (SC)
- net VSC8: now reaches U29.64 (SC)
- net VSC6: now reaches U37.64 (SC)
- net VSC6: now also U27.64 (SC)
- net VSC7: now reaches U28.64 (SC)
- net VSC7: now also U38.64 (SC)
- net VSC2: now reaches U35.64 (SC)
- net VSC2: now also U25.64 (SC)
- net VSC4: now reaches U56.64 (SC)
- net VSC4: now also U48.64 (SC)
- net VSC3: now reaches U26.64 (SC)
- net VSC3: now also U36.64 (SC)
- no-connect marks 0 -> 16
Other:
- note removed: "all chips"

Commit message: add test points
Parts:
- added TP288: U25_0, hp16717:HP_TP30, symbol Connector:TestPoint_Alt
- added TP289: U25_1, hp16717:HP_TP30, symbol Connector:TestPoint_Alt
- added TP290: U25_2, hp16717:HP_TP30, symbol Connector:TestPoint_Alt
- added TP291: U25_3, hp16717:HP_TP30, symbol Connector:TestPoint_Alt
- added TP292: U25_4, hp16717:HP_TP30, symbol Connector:TestPoint_Alt
- added TP293: U25_5, hp16717:HP_TP30, symbol Connector:TestPoint_Alt
- added TP294: U25_6, hp16717:HP_TP30, symbol Connector:TestPoint_Alt
- added TP295: U25_7, hp16717:HP_TP30, symbol Connector:TestPoint_Alt
- added TP296: U25_8, hp16717:HP_TP30, symbol Connector:TestPoint_Alt
- added TP297: U25_9, hp16717:HP_TP30, symbol Connector:TestPoint_Alt
- added TP298: U25_10, hp16717:HP_TP30, symbol Connector:TestPoint_Alt
- added TP299: U25_11, hp16717:HP_TP30, symbol Connector:TestPoint_Alt
- added TP300: U25_12, hp16717:HP_TP30, symbol Connector:TestPoint_Alt
- added TP301: U25_13, hp16717:HP_TP30, symbol Connector:TestPoint_Alt
- added TP302: U25_14, hp16717:HP_TP30, symbol Connector:TestPoint_Alt
- added TP303: U25_15, hp16717:HP_TP30, symbol Connector:TestPoint_Alt
- added TP304: VSC0, hp16717:HP_TP30, symbol Connector:TestPoint_Alt
- added TP305: VSC1, hp16717:HP_TP30, symbol Connector:TestPoint_Alt
- added TP306: VSC2, hp16717:HP_TP30, symbol Connector:TestPoint_Alt
- added TP307: VSC3, hp16717:HP_TP30, symbol Connector:TestPoint_Alt
- added TP308: U35_0, hp16717:HP_TP30, symbol Connector:TestPoint_Alt
- added TP309: U35_1, hp16717:HP_TP30, symbol Connector:TestPoint_Alt
- added TP310: U35_2, hp16717:HP_TP30, symbol Connector:TestPoint_Alt
- added TP311: U35_3, hp16717:HP_TP30, symbol Connector:TestPoint_Alt
- added TP312: U35_4, hp16717:HP_TP30, symbol Connector:TestPoint_Alt
- added TP313: U35_5, hp16717:HP_TP30, symbol Connector:TestPoint_Alt
- added TP314: U35_6, hp16717:HP_TP30, symbol Connector:TestPoint_Alt
- added TP315: U35_7, hp16717:HP_TP30, symbol Connector:TestPoint_Alt
- added TP316: U35_8, hp16717:HP_TP30, symbol Connector:TestPoint_Alt
- added TP317: U35_9, hp16717:HP_TP30, symbol Connector:TestPoint_Alt
- added TP318: U35_10, hp16717:HP_TP30, symbol Connector:TestPoint_Alt
- added TP319: U35_11, hp16717:HP_TP30, symbol Connector:TestPoint_Alt
- added TP320: U35_12, hp16717:HP_TP30, symbol Connector:TestPoint_Alt
- added TP321: U35_13, hp16717:HP_TP30, symbol Connector:TestPoint_Alt
- added TP322: U35_14, hp16717:HP_TP30, symbol Connector:TestPoint_Alt
- added TP323: U35_15, hp16717:HP_TP30, symbol Connector:TestPoint_Alt
- added TP324: U46_0, hp16717:HP_TP30, symbol Connector:TestPoint_Alt
- added TP325: U46_1, hp16717:HP_TP30, symbol Connector:TestPoint_Alt
- added TP326: U46_2, hp16717:HP_TP30, symbol Connector:TestPoint_Alt
- added TP327: U46_3, hp16717:HP_TP30, symbol Connector:TestPoint_Alt
- added TP328: U46_4, hp16717:HP_TP30, symbol Connector:TestPoint_Alt
- added TP329: U46_5, hp16717:HP_TP30, symbol Connector:TestPoint_Alt
- added TP330: U46_6, hp16717:HP_TP30, symbol Connector:TestPoint_Alt
- added TP331: U46_7, hp16717:HP_TP30, symbol Connector:TestPoint_Alt
- added TP332: U46_8, hp16717:HP_TP30, symbol Connector:TestPoint_Alt
- added TP333: U46_9, hp16717:HP_TP30, symbol Connector:TestPoint_Alt
- added TP334: U46_10, hp16717:HP_TP30, symbol Connector:TestPoint_Alt
- added TP335: U46_11, hp16717:HP_TP30, symbol Connector:TestPoint_Alt
- added TP336: U46_12, hp16717:HP_TP30, symbol Connector:TestPoint_Alt
- added TP337: U46_13, hp16717:HP_TP30, symbol Connector:TestPoint_Alt
- added TP338: U46_14, hp16717:HP_TP30, symbol Connector:TestPoint_Alt
- added TP339: U46_15, hp16717:HP_TP30, symbol Connector:TestPoint_Alt
- added TP340: U54_0, hp16717:HP_TP30, symbol Connector:TestPoint_Alt
- added TP341: U54_1, hp16717:HP_TP30, symbol Connector:TestPoint_Alt
- added TP342: U54_2, hp16717:HP_TP30, symbol Connector:TestPoint_Alt
- added TP343: U54_3, hp16717:HP_TP30, symbol Connector:TestPoint_Alt
- added TP344: U54_4, hp16717:HP_TP30, symbol Connector:TestPoint_Alt
- added TP345: U54_5, hp16717:HP_TP30, symbol Connector:TestPoint_Alt
- added TP346: U54_6, hp16717:HP_TP30, symbol Connector:TestPoint_Alt
- added TP347: U54_7, hp16717:HP_TP30, symbol Connector:TestPoint_Alt
- added TP348: U54_8, hp16717:HP_TP30, symbol Connector:TestPoint_Alt
- added TP349: U54_9, hp16717:HP_TP30, symbol Connector:TestPoint_Alt
- added TP350: U54_10, hp16717:HP_TP30, symbol Connector:TestPoint_Alt
- added TP351: U54_11, hp16717:HP_TP30, symbol Connector:TestPoint_Alt
- added TP352: U54_12, hp16717:HP_TP30, symbol Connector:TestPoint_Alt
- added TP353: U54_13, hp16717:HP_TP30, symbol Connector:TestPoint_Alt
- added TP354: U54_14, hp16717:HP_TP30, symbol Connector:TestPoint_Alt
- added TP355: U54_15, hp16717:HP_TP30, symbol Connector:TestPoint_Alt
- added TP356: U27_0, hp16717:HP_TP30, symbol Connector:TestPoint_Alt
- added TP357: U27_1, hp16717:HP_TP30, symbol Connector:TestPoint_Alt
- added TP358: U27_2, hp16717:HP_TP30, symbol Connector:TestPoint_Alt
- added TP359: U27_3, hp16717:HP_TP30, symbol Connector:TestPoint_Alt
- added TP360: U27_4, hp16717:HP_TP30, symbol Connector:TestPoint_Alt
- added TP361: U27_5, hp16717:HP_TP30, symbol Connector:TestPoint_Alt
- added TP362: U27_6, hp16717:HP_TP30, symbol Connector:TestPoint_Alt
- added TP363: U27_7, hp16717:HP_TP30, symbol Connector:TestPoint_Alt
- added TP364: U27_8, hp16717:HP_TP30, symbol Connector:TestPoint_Alt
- added TP365: U27_9, hp16717:HP_TP30, symbol Connector:TestPoint_Alt
- added TP366: U27_10, hp16717:HP_TP30, symbol Connector:TestPoint_Alt
- added TP367: U27_11, hp16717:HP_TP30, symbol Connector:TestPoint_Alt
- added TP368: U27_12, hp16717:HP_TP30, symbol Connector:TestPoint_Alt
- added TP369: U27_13, hp16717:HP_TP30, symbol Connector:TestPoint_Alt
- added TP370: U27_14, hp16717:HP_TP30, symbol Connector:TestPoint_Alt
- added TP371: U27_15, hp16717:HP_TP30, symbol Connector:TestPoint_Alt
- added TP372: U37_0, hp16717:HP_TP30, symbol Connector:TestPoint_Alt
- added TP373: U37_1, hp16717:HP_TP30, symbol Connector:TestPoint_Alt
- added TP374: U37_2, hp16717:HP_TP30, symbol Connector:TestPoint_Alt
- added TP375: U37_3, hp16717:HP_TP30, symbol Connector:TestPoint_Alt
- added TP376: U37_4, hp16717:HP_TP30, symbol Connector:TestPoint_Alt
- added TP377: U37_5, hp16717:HP_TP30, symbol Connector:TestPoint_Alt
- added TP378: U37_6, hp16717:HP_TP30, symbol Connector:TestPoint_Alt
- added TP379: U37_7, hp16717:HP_TP30, symbol Connector:TestPoint_Alt
- added TP380: U37_8, hp16717:HP_TP30, symbol Connector:TestPoint_Alt
- added TP381: U37_9, hp16717:HP_TP30, symbol Connector:TestPoint_Alt
- added TP382: U37_10, hp16717:HP_TP30, symbol Connector:TestPoint_Alt
- added TP383: U37_11, hp16717:HP_TP30, symbol Connector:TestPoint_Alt
- added TP384: U37_12, hp16717:HP_TP30, symbol Connector:TestPoint_Alt
- added TP385: U37_13, hp16717:HP_TP30, symbol Connector:TestPoint_Alt
- added TP386: U37_14, hp16717:HP_TP30, symbol Connector:TestPoint_Alt
- added TP387: U37_15, hp16717:HP_TP30, symbol Connector:TestPoint_Alt
- added TP388: U48_0, hp16717:HP_TP30, symbol Connector:TestPoint_Alt
- added TP389: U48_1, hp16717:HP_TP30, symbol Connector:TestPoint_Alt
- added TP390: U48_2, hp16717:HP_TP30, symbol Connector:TestPoint_Alt
- added TP391: U48_3, hp16717:HP_TP30, symbol Connector:TestPoint_Alt
- added TP392: U48_4, hp16717:HP_TP30, symbol Connector:TestPoint_Alt
- added TP393: U48_5, hp16717:HP_TP30, symbol Connector:TestPoint_Alt
- added TP394: U48_6, hp16717:HP_TP30, symbol Connector:TestPoint_Alt
- added TP395: U48_7, hp16717:HP_TP30, symbol Connector:TestPoint_Alt
- added TP396: U48_8, hp16717:HP_TP30, symbol Connector:TestPoint_Alt
- added TP397: U48_9, hp16717:HP_TP30, symbol Connector:TestPoint_Alt
- added TP398: U48_10, hp16717:HP_TP30, symbol Connector:TestPoint_Alt
- added TP399: U48_11, hp16717:HP_TP30, symbol Connector:TestPoint_Alt
- added TP400: U48_12, hp16717:HP_TP30, symbol Connector:TestPoint_Alt
- added TP401: U48_13, hp16717:HP_TP30, symbol Connector:TestPoint_Alt
- added TP402: U48_14, hp16717:HP_TP30, symbol Connector:TestPoint_Alt
- added TP403: U48_15, hp16717:HP_TP30, symbol Connector:TestPoint_Alt
- added TP404: U56_0, hp16717:HP_TP30, symbol Connector:TestPoint_Alt
- added TP405: U56_1, hp16717:HP_TP30, symbol Connector:TestPoint_Alt
- added TP406: U56_2, hp16717:HP_TP30, symbol Connector:TestPoint_Alt
- added TP407: U56_3, hp16717:HP_TP30, symbol Connector:TestPoint_Alt
- added TP408: U56_4, hp16717:HP_TP30, symbol Connector:TestPoint_Alt
- added TP409: U56_5, hp16717:HP_TP30, symbol Connector:TestPoint_Alt
- added TP410: U56_6, hp16717:HP_TP30, symbol Connector:TestPoint_Alt
- added TP411: U56_7, hp16717:HP_TP30, symbol Connector:TestPoint_Alt
- added TP412: U56_8, hp16717:HP_TP30, symbol Connector:TestPoint_Alt
- added TP413: U56_9, hp16717:HP_TP30, symbol Connector:TestPoint_Alt
- added TP414: U56_10, hp16717:HP_TP30, symbol Connector:TestPoint_Alt
- added TP415: U56_11, hp16717:HP_TP30, symbol Connector:TestPoint_Alt
- added TP416: U56_12, hp16717:HP_TP30, symbol Connector:TestPoint_Alt
- added TP417: U56_13, hp16717:HP_TP30, symbol Connector:TestPoint_Alt
- added TP418: U56_14, hp16717:HP_TP30, symbol Connector:TestPoint_Alt
- added TP419: U56_15, hp16717:HP_TP30, symbol Connector:TestPoint_Alt
- added TP420: U29_0, hp16717:HP_TP30, symbol Connector:TestPoint_Alt
- added TP423: U29_3, hp16717:HP_TP30, symbol Connector:TestPoint_Alt
- added TP425: U29_5, hp16717:HP_TP30, symbol Connector:TestPoint_Alt
- added TP427: U29_7, hp16717:HP_TP30, symbol Connector:TestPoint_Alt
- added TP428: U29_8, hp16717:HP_TP30, symbol Connector:TestPoint_Alt
- added TP429: U29_9, hp16717:HP_TP30, symbol Connector:TestPoint_Alt
- added TP430: U29_10, hp16717:HP_TP30, symbol Connector:TestPoint_Alt
- added TP431: U29_11, hp16717:HP_TP30, symbol Connector:TestPoint_Alt
- added TP432: U29_12, hp16717:HP_TP30, symbol Connector:TestPoint_Alt
- added TP433: U29_13, hp16717:HP_TP30, symbol Connector:TestPoint_Alt
- added TP434: U29_14, hp16717:HP_TP30, symbol Connector:TestPoint_Alt
- added TP435: U29_15, hp16717:HP_TP30, symbol Connector:TestPoint_Alt
- added TP436, TP437, TP438, TP439, TP440, TP441, TP442, TP443, TP444, TP455, TP456, TP457, TP458, TP463, TP464, TP465: +5V, hp16717:HP_TP30, symbol Connector:TestPoint_Alt
- added TP445, TP446, TP447, TP448, TP449, TP450, TP451, TP452, TP453, TP454, TP459, TP460, TP461, TP462, TP466, TP467, TP468, TP469, TP470: GND, hp16717:HP_TP30, symbol Connector:TestPoint_Alt
- added TP471: VSC4, hp16717:HP_TP30, symbol Connector:TestPoint_Alt
- added TP472: VSC5, hp16717:HP_TP30, symbol Connector:TestPoint_Alt
- added TP473: VSC6, hp16717:HP_TP30, symbol Connector:TestPoint_Alt
- added TP474: VSC7, hp16717:HP_TP30, symbol Connector:TestPoint_Alt
- added TP475: VSC8, hp16717:HP_TP30, symbol Connector:TestPoint_Alt
Connections:
- net +5V: now also TP436.1, TP437.1, TP438.1, TP439.1, TP440.1, TP441.1, TP442.1, TP443.1, TP444.1, TP455.1, TP456.1, TP457.1, TP458.1, TP463.1, TP464.1, TP465.1
- net GND: now also TP445.1, TP446.1, TP447.1, TP448.1, TP449.1, TP450.1, TP451.1, TP452.1, TP453.1, TP454.1, TP459.1, TP460.1, TP461.1, TP462.1, TP466.1, TP467.1, TP468.1, TP469.1, TP470.1
- net U25_0: now also TP288.1
- net U25_1: now also TP289.1
- net U25_10: now also TP298.1
- net U25_11: now also TP299.1
- net U25_12: now also TP300.1
- net U25_13: now also TP301.1
- net U25_14: now also TP302.1
- net U25_15: now also TP303.1
- net U25_2: now also TP290.1
- net U25_3: now also TP291.1
- net U25_4: now also TP292.1
- net U25_5: now also TP293.1
- net U25_6: now also TP294.1
- net U25_7: now also TP295.1
- net U25_8: now also TP296.1
- net U25_9: now also TP297.1
- net U27_0: now also TP356.1
- net U27_1: now also TP357.1
- net U27_10: now also TP366.1
- net U27_11: now also TP367.1
- net U27_12: now also TP368.1
- net U27_13: now also TP369.1
- net U27_14: now also TP370.1
- net U27_15: now also TP371.1
- net U27_2: now also TP358.1
- net U27_3: now also TP359.1
- net U27_4: now also TP360.1
- net U27_5: now also TP361.1
- net U27_6: now also TP362.1
- net U27_7: now also TP363.1
- net U27_8: now also TP364.1
- net U27_9: now also TP365.1
- net U29_0: now also TP420.1
- net U29_10: now also TP430.1
- net U29_11: now also TP431.1
- net U29_12: now also TP432.1
- net U29_13: now also TP433.1
- net U29_14: now also TP434.1
- net U29_15: now also TP435.1
- net U29_3: now also TP423.1
- net U29_5: now also TP425.1
- net U29_7: now also TP427.1
- net U29_8: now also TP428.1
- net U29_9: now also TP429.1
- net U35_0: now also TP308.1
- net U35_1: now also TP309.1
- net U35_10: now also TP318.1
- net U35_11: now also TP319.1
- net U35_12: now also TP320.1
- net U35_13: now also TP321.1
- net U35_14: now also TP322.1
- net U35_15: now also TP323.1
- net U35_2: now also TP310.1
- net U35_3: now also TP311.1
- net U35_4: now also TP312.1
- net U35_5: now also TP313.1
- net U35_6: now also TP314.1
- net U35_7: now also TP315.1
- net U35_8: now also TP316.1
- net U35_9: now also TP317.1
- net U37_0: now also TP372.1
- net U37_1: now also TP373.1
- net U37_10: now also TP382.1
- net U37_11: now also TP383.1
- net U37_12: now also TP384.1
- net U37_13: now also TP385.1
- net U37_14: now also TP386.1
- net U37_15: now also TP387.1
- net U37_2: now also TP374.1
- net U37_3: now also TP375.1
- net U37_4: now also TP376.1
- net U37_5: now also TP377.1
- net U37_6: now also TP378.1
- net U37_7: now also TP379.1
- net U37_8: now also TP380.1
- net U37_9: now also TP381.1
- net U46_0: now also TP324.1
- net U46_1: now also TP325.1
- net U46_10: now also TP334.1
- net U46_11: now also TP335.1
- net U46_12: now also TP336.1
- net U46_13: now also TP337.1
- net U46_14: now also TP338.1
- net U46_15: now also TP339.1
- net U46_2: now also TP326.1
- net U46_3: now also TP327.1
- net U46_4: now also TP328.1
- net U46_5: now also TP329.1
- net U46_6: now also TP330.1
- net U46_7: now also TP331.1
- net U46_8: now also TP332.1
- net U46_9: now also TP333.1
- net U48_0: now also TP388.1
- net U48_1: now also TP389.1
- net U48_10: now also TP398.1
- net U48_11: now also TP399.1
- net U48_12: now also TP400.1
- net U48_13: now also TP401.1
- net U48_14: now also TP402.1
- net U48_15: now also TP403.1
- net U48_2: now also TP390.1
- net U48_3: now also TP391.1
- net U48_4: now also TP392.1
- net U48_5: now also TP393.1
- net U48_6: now also TP394.1
- net U48_7: now also TP395.1
- net U48_8: now also TP396.1
- net U48_9: now also TP397.1
- net U54_0: now also TP340.1
- net U54_1: now also TP341.1
- net U54_10: now also TP350.1
- net U54_11: now also TP351.1
- net U54_12: now also TP352.1
- net U54_13: now also TP353.1
- net U54_14: now also TP354.1
- net U54_15: now also TP355.1
- net U54_2: now also TP342.1
- net U54_3: now also TP343.1
- net U54_4: now also TP344.1
- net U54_5: now also TP345.1
- net U54_6: now also TP346.1
- net U54_7: now also TP347.1
- net U54_8: now also TP348.1
- net U54_9: now also TP349.1
- net U56_0: now also TP404.1
- net U56_1: now also TP405.1
- net U56_10: now also TP414.1
- net U56_11: now also TP415.1
- net U56_12: now also TP416.1
- net U56_13: now also TP417.1
- net U56_14: now also TP418.1
- net U56_15: now also TP419.1
- net U56_2: now also TP406.1
- net U56_3: now also TP407.1
- net U56_4: now also TP408.1
- net U56_5: now also TP409.1
- net U56_6: now also TP410.1
- net U56_7: now also TP411.1
- net U56_8: now also TP412.1
- net U56_9: now also TP413.1
- net VSC0: now also TP304.1
- net VSC1: now also TP305.1
- net VSC2: now also TP306.1
- net VSC3: now also TP307.1
- net VSC4: now also TP471.1
- net VSC5: now also TP472.1
- net VSC6: now also TP473.1
- net VSC7: now also TP474.1
- net VSC8: now also TP475.1
